File: my-keeb.kicad_pcb (KiCad board)
At the start: 2 copper layers, 360 x 170 mm, 183 parts, among them SW10 SW_Push, SW11 SW_Push, SW12 SW_Push, SW13 SW_Push, SW14 SW_Push, SW16 SW_Push, SW17 SW_Push, SW18 SW_Push, SW19 SW_Push, SW2 SW_Push, SW20 SW_Push, SW21 SW_Push, SW22 SW_Push, SW23 SW_Push, SW24 SW_Push, SW25 SW_Push, SW26 SW_Push, SW27 SW_Push, SW29 SW_Push, SW3 SW_Push, SW30 SW_Push, SW31 SW_Push, SW32 SW_Push, SW33 SW_Push, SW34 SW_Push, SW35 SW_Push, SW36 SW_Push, SW37 SW_Push, SW38 SW_Push, SW39 SW_Push, SW4 SW_Push, SW40 SW_Push, SW41 SW_Push, SW42 SW_Push, SW43 SW_Push, SW44 SW_Push, SW45 SW_Push, SW46 SW_Push, SW47 SW_Push, SW48 SW_Push, SW49 SW_Push, SW5 SW_Push, SW50 SW_Push, SW51 SW_Push, SW52 SW_Push, SW53 SW_Push, SW54 SW_Push, SW55 SW_Push, SW57 SW_Push, SW58 SW_Push, SW6 SW_Push, SW60 SW_Push, SW61 SW_Push, SW62 SW_Push, SW63 SW_Push, SW64 SW_Push, SW65 SW_Push, SW66 SW_Push, SW67 SW_Push, SW68 SW_Push, SW69 SW_Push, SW7 SW_Push, SW71 SW_Push, SW72 SW_Push, SW73 SW_Push, SW74 SW_Push, SW75 SW_Push, SW77 SW_Push, SW79 SW_Push, SW8 SW_Push, SW80 SW_Push, SW81 SW_Push, SW82 SW_Push, SW84 SW_Push, SW85 SW_Push, SW86 SW_Push, SW87 SW_Push, SW88 SW_Push, SW89 SW_Push, SW9 SW_Push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

Commit message: Add files via upload
Parts:
- removed D75, D84, D85: 1N4148, Diode_THT:D_DO-35_SOD27_P7.62mm_Horizontal
- removed S2: MX_stab, PCM_marbastlib-mx:STAB_MX_P_2u
- removed S5, S6: MX_stab, my-keeb:STAB_MX_P_2u
- removed SW75, SW84, SW85: SW_Push, PCM_marbastlib-mx:SW_MX_1u
- added D94: 1N4148, Diode_THT:D_DO-35_SOD27_P7.62mm_Horizontal, B.Cu at (340.3, 106.5)
- added D95: 1N4148, Diode_THT:D_DO-35_SOD27_P7.62mm_Horizontal, B.Cu at (358.8, 108.0)
- added MH1: MountingHole_3.048mm, MountingHole:MountingHole_3.048mm, F.Cu at (93.5, 128.3)
- added MH2: MountingHole_3.048mm, MountingHole:MountingHole_3.048mm, F.Cu at (193.5, 128.3)
- added MH3: MountingHole_3.9878mm, MountingHole:MountingHole_3.9878mm, F.Cu at (93.5, 143.5)
- added MH4: MountingHole_3.9878mm, MountingHole:MountingHole_3.9878mm, F.Cu at (193.5, 143.5)
- added RGB1: SK6812MINI-E, my-keeb:LED_SK6812MINI-E_3.2x2.8mm_P1.5mm_ReverseMount, B.Cu at (206.0, 44.2)
- added RGB10: SK6812MINI-E, my-keeb:LED_SK6812MINI-E_3.2x2.8mm_P1.5mm_ReverseMount, B.Cu at (234.6, 44.2)
- added RGB11: SK6812MINI-E, my-keeb:LED_SK6812MINI-E_3.2x2.8mm_P1.5mm_ReverseMount, B.Cu at (253.6, 44.2)
- added RGB12: SK6812MINI-E, my-keeb:LED_SK6812MINI-E_3.2x2.8mm_P1.5mm_ReverseMount, B.Cu at (272.6, 44.2)
- added RGB13: SK6812MINI-E, my-keeb:LED_SK6812MINI-E_3.2x2.8mm_P1.5mm_ReverseMount, B.Cu at (291.7, 44.2)
- added RGB14: SK6812MINI-E, my-keeb:LED_SK6812MINI-E_3.2x2.8mm_P1.5mm_ReverseMount, B.Cu at (25.0, 63.2)
- added RGB15: SK6812MINI-E, my-keeb:LED_SK6812MINI-E_3.2x2.8mm_P1.5mm_ReverseMount, B.Cu at (44.0, 63.2)
- added RGB16: SK6812MINI-E, my-keeb:LED_SK6812MINI-E_3.2x2.8mm_P1.5mm_ReverseMount, B.Cu at (63.1, 63.2)
- added RGB17: SK6812MINI-E, my-keeb:LED_SK6812MINI-E_3.2x2.8mm_P1.5mm_ReverseMount, B.Cu at (82.2, 63.2)
- added RGB18: SK6812MINI-E, my-keeb:LED_SK6812MINI-E_3.2x2.8mm_P1.5mm_ReverseMount, B.Cu at (101.2, 63.2)
- added RGB19: SK6812MINI-E, my-keeb:LED_SK6812MINI-E_3.2x2.8mm_P1.5mm_ReverseMount, B.Cu at (120.2, 63.2)
- added RGB2: SK6812MINI-E, my-keeb:LED_SK6812MINI-E_3.2x2.8mm_P1.5mm_ReverseMount, B.Cu at (25.0, 44.2)
- added RGB20: SK6812MINI-E, my-keeb:LED_SK6812MINI-E_3.2x2.8mm_P1.5mm_ReverseMount, B.Cu at (139.3, 63.2)
- added RGB21: SK6812MINI-E, my-keeb:LED_SK6812MINI-E_3.2x2.8mm_P1.5mm_ReverseMount, B.Cu at (158.3, 63.2)
- added RGB22: SK6812MINI-E, my-keeb:LED_SK6812MINI-E_3.2x2.8mm_P1.5mm_ReverseMount, B.Cu at (177.4, 63.2)
- added RGB23: SK6812MINI-E, my-keeb:LED_SK6812MINI-E_3.2x2.8mm_P1.5mm_ReverseMount, B.Cu at (196.4, 63.2)
- added RGB24: SK6812MINI-E, my-keeb:LED_SK6812MINI-E_3.2x2.8mm_P1.5mm_ReverseMount, B.Cu at (215.5, 63.2)
- added RGB25: SK6812MINI-E, my-keeb:LED_SK6812MINI-E_3.2x2.8mm_P1.5mm_ReverseMount, B.Cu at (234.6, 63.2)
- added RGB26: SK6812MINI-E, my-keeb:LED_SK6812MINI-E_3.2x2.8mm_P1.5mm_ReverseMount, B.Cu at (253.6, 63.2)
- added RGB27: SK6812MINI-E, my-keeb:LED_SK6812MINI-E_3.2x2.8mm_P1.5mm_ReverseMount, B.Cu at (282.2, 63.2)
- added RGB28: SK6812MINI-E, my-keeb:LED_SK6812MINI-E_3.2x2.8mm_P1.5mm_ReverseMount, B.Cu at (336.5, 63.2)
- added RGB29: SK6812MINI-E, my-keeb:LED_SK6812MINI-E_3.2x2.8mm_P1.5mm_ReverseMount, B.Cu at (355.6, 63.2)
- added RGB3: SK6812MINI-E, my-keeb:LED_SK6812MINI-E_3.2x2.8mm_P1.5mm_ReverseMount, B.Cu at (63.1, 44.2)
- added RGB30: SK6812MINI-E, my-keeb:LED_SK6812MINI-E_3.2x2.8mm_P1.5mm_ReverseMount, B.Cu at (29.7, 82.2)
- added RGB31: SK6812MINI-E, my-keeb:LED_SK6812MINI-E_3.2x2.8mm_P1.5mm_ReverseMount, B.Cu at (53.6, 82.2)
- added RGB32: SK6812MINI-E, my-keeb:LED_SK6812MINI-E_3.2x2.8mm_P1.5mm_ReverseMount, B.Cu at (72.6, 82.2)
- added RGB33: SK6812MINI-E, my-keeb:LED_SK6812MINI-E_3.2x2.8mm_P1.5mm_ReverseMount, B.Cu at (91.7, 82.2)
- added RGB34: SK6812MINI-E, my-keeb:LED_SK6812MINI-E_3.2x2.8mm_P1.5mm_ReverseMount, B.Cu at (110.7, 82.2)
- added RGB35: SK6812MINI-E, my-keeb:LED_SK6812MINI-E_3.2x2.8mm_P1.5mm_ReverseMount, B.Cu at (129.8, 82.2)
- added RGB36: SK6812MINI-E, my-keeb:LED_SK6812MINI-E_3.2x2.8mm_P1.5mm_ReverseMount, B.Cu at (148.8, 82.2)
- added RGB37: SK6812MINI-E, my-keeb:LED_SK6812MINI-E_3.2x2.8mm_P1.5mm_ReverseMount, B.Cu at (167.9, 82.2)
- added RGB38: SK6812MINI-E, my-keeb:LED_SK6812MINI-E_3.2x2.8mm_P1.5mm_ReverseMount, B.Cu at (186.9, 82.2)
- added RGB39: SK6812MINI-E, my-keeb:LED_SK6812MINI-E_3.2x2.8mm_P1.5mm_ReverseMount, B.Cu at (206.0, 82.2)
- added RGB4: SK6812MINI-E, my-keeb:LED_SK6812MINI-E_3.2x2.8mm_P1.5mm_ReverseMount, B.Cu at (82.2, 44.2)
- added RGB40: SK6812MINI-E, my-keeb:LED_SK6812MINI-E_3.2x2.8mm_P1.5mm_ReverseMount, B.Cu at (225.0, 82.2)
- added RGB41: SK6812MINI-E, my-keeb:LED_SK6812MINI-E_3.2x2.8mm_P1.5mm_ReverseMount, B.Cu at (244.1, 82.2)
- added RGB42: SK6812MINI-E, my-keeb:LED_SK6812MINI-E_3.2x2.8mm_P1.5mm_ReverseMount, B.Cu at (263.1, 82.2)
- added RGB43: SK6812MINI-E, my-keeb:LED_SK6812MINI-E_3.2x2.8mm_P1.5mm_ReverseMount, B.Cu at (286.9, 82.2)
- added RGB44: SK6812MINI-E, my-keeb:LED_SK6812MINI-E_3.2x2.8mm_P1.5mm_ReverseMount, B.Cu at (336.5, 82.2)
- added RGB45: SK6812MINI-E, my-keeb:LED_SK6812MINI-E_3.2x2.8mm_P1.5mm_ReverseMount, B.Cu at (355.6, 82.2)
- added RGB46: SK6812MINI-E, my-keeb:LED_SK6812MINI-E_3.2x2.8mm_P1.5mm_ReverseMount, B.Cu at (58.3, 101.2)
- added RGB47: SK6812MINI-E, my-keeb:LED_SK6812MINI-E_3.2x2.8mm_P1.5mm_ReverseMount, B.Cu at (77.4, 101.2)
- added RGB48: SK6812MINI-E, my-keeb:LED_SK6812MINI-E_3.2x2.8mm_P1.5mm_ReverseMount, B.Cu at (96.4, 101.2)
- added RGB49: SK6812MINI-E, my-keeb:LED_SK6812MINI-E_3.2x2.8mm_P1.5mm_ReverseMount, B.Cu at (115.5, 101.2)
- added RGB5: SK6812MINI-E, my-keeb:LED_SK6812MINI-E_3.2x2.8mm_P1.5mm_ReverseMount, B.Cu at (101.2, 44.2)
- added RGB50: SK6812MINI-E, my-keeb:LED_SK6812MINI-E_3.2x2.8mm_P1.5mm_ReverseMount, B.Cu at (134.5, 101.2)
- added RGB51: SK6812MINI-E, my-keeb:LED_SK6812MINI-E_3.2x2.8mm_P1.5mm_ReverseMount, B.Cu at (153.6, 101.2)
- added RGB52: SK6812MINI-E, my-keeb:LED_SK6812MINI-E_3.2x2.8mm_P1.5mm_ReverseMount, B.Cu at (172.6, 101.2)
- added RGB53: SK6812MINI-E, my-keeb:LED_SK6812MINI-E_3.2x2.8mm_P1.5mm_ReverseMount, B.Cu at (191.7, 101.2)
- added RGB54: SK6812MINI-E, my-keeb:LED_SK6812MINI-E_3.2x2.8mm_P1.5mm_ReverseMount, B.Cu at (210.7, 101.2)
- added RGB55: SK6812MINI-E, my-keeb:LED_SK6812MINI-E_3.2x2.8mm_P1.5mm_ReverseMount, B.Cu at (229.8, 101.2)
- added RGB56: SK6812MINI-E, my-keeb:LED_SK6812MINI-E_3.2x2.8mm_P1.5mm_ReverseMount, B.Cu at (248.8, 101.2)
- added RGB57: SK6812MINI-E, my-keeb:LED_SK6812MINI-E_3.2x2.8mm_P1.5mm_ReverseMount, B.Cu at (279.8, 101.2)
- added RGB58: SK6812MINI-E, my-keeb:LED_SK6812MINI-E_3.2x2.8mm_P1.5mm_ReverseMount, B.Cu at (32.1, 101.2)
- added RGB59: SK6812MINI-E, my-keeb:LED_SK6812MINI-E_3.2x2.8mm_P1.5mm_ReverseMount, B.Cu at (67.9, 120.2)
- added RGB6: SK6812MINI-E, my-keeb:LED_SK6812MINI-E_3.2x2.8mm_P1.5mm_ReverseMount, B.Cu at (120.2, 44.2)
- added RGB60: SK6812MINI-E, my-keeb:LED_SK6812MINI-E_3.2x2.8mm_P1.5mm_ReverseMount, B.Cu at (86.9, 120.2)
- added RGB61: SK6812MINI-E, my-keeb:LED_SK6812MINI-E_3.2x2.8mm_P1.5mm_ReverseMount, B.Cu at (106.0, 120.2)
- added RGB62: SK6812MINI-E, my-keeb:LED_SK6812MINI-E_3.2x2.8mm_P1.5mm_ReverseMount, B.Cu at (125.0, 120.2)
- added RGB63: SK6812MINI-E, my-keeb:LED_SK6812MINI-E_3.2x2.8mm_P1.5mm_ReverseMount, B.Cu at (144.1, 120.2)
- added RGB64: SK6812MINI-E, my-keeb:LED_SK6812MINI-E_3.2x2.8mm_P1.5mm_ReverseMount, B.Cu at (163.1, 120.2)
- added RGB65: SK6812MINI-E, my-keeb:LED_SK6812MINI-E_3.2x2.8mm_P1.5mm_ReverseMount, B.Cu at (182.2, 120.2)
- added RGB66: SK6812MINI-E, my-keeb:LED_SK6812MINI-E_3.2x2.8mm_P1.5mm_ReverseMount, B.Cu at (201.2, 120.2)
- added RGB67: SK6812MINI-E, my-keeb:LED_SK6812MINI-E_3.2x2.8mm_P1.5mm_ReverseMount, B.Cu at (220.3, 120.2)
- added RGB68: SK6812MINI-E, my-keeb:LED_SK6812MINI-E_3.2x2.8mm_P1.5mm_ReverseMount, B.Cu at (239.3, 120.2)
- added RGB69: SK6812MINI-E, my-keeb:LED_SK6812MINI-E_3.2x2.8mm_P1.5mm_ReverseMount, B.Cu at (275.0, 120.2)
- added RGB7: SK6812MINI-E, my-keeb:LED_SK6812MINI-E_3.2x2.8mm_P1.5mm_ReverseMount, B.Cu at (148.8, 44.2)
- added RGB70: SK6812MINI-E, my-keeb:LED_SK6812MINI-E_3.2x2.8mm_P1.5mm_ReverseMount, B.Cu at (336.5, 120.2)
- added RGB71: SK6812MINI-E, my-keeb:LED_SK6812MINI-E_3.2x2.8mm_P1.5mm_ReverseMount, B.Cu at (27.4, 139.2)
- added RGB72: SK6812MINI-E, my-keeb:LED_SK6812MINI-E_3.2x2.8mm_P1.5mm_ReverseMount, B.Cu at (51.2, 139.2)
- added RGB73: SK6812MINI-E, my-keeb:LED_SK6812MINI-E_3.2x2.8mm_P1.5mm_ReverseMount, B.Cu at (75.0, 139.2)
- added RGB74: SK6812MINI-E, my-keeb:LED_SK6812MINI-E_3.2x2.8mm_P1.5mm_ReverseMount, B.Cu at (36.9, 120.2)
- added RGB75: SK6812MINI-E, my-keeb:LED_SK6812MINI-E_3.2x2.8mm_P1.5mm_ReverseMount, B.Cu at (146.4, 139.2)
- added RGB76: SK6812MINI-E, my-keeb:LED_SK6812MINI-E_3.2x2.8mm_P1.5mm_ReverseMount, B.Cu at (217.9, 139.2)
- added RGB77: SK6812MINI-E, my-keeb:LED_SK6812MINI-E_3.2x2.8mm_P1.5mm_ReverseMount, B.Cu at (241.7, 139.2)
- added RGB78: SK6812MINI-E, my-keeb:LED_SK6812MINI-E_3.2x2.8mm_P1.5mm_ReverseMount, B.Cu at (265.5, 139.2)
- added RGB79: SK6812MINI-E, my-keeb:LED_SK6812MINI-E_3.2x2.8mm_P1.5mm_ReverseMount, B.Cu at (289.3, 139.2)
- added RGB8: SK6812MINI-E, my-keeb:LED_SK6812MINI-E_3.2x2.8mm_P1.5mm_ReverseMount, B.Cu at (167.9, 44.2)
- added RGB80: SK6812MINI-E, my-keeb:LED_SK6812MINI-E_3.2x2.8mm_P1.5mm_ReverseMount, B.Cu at (317.4, 139.2)
- added RGB81: SK6812MINI-E, my-keeb:LED_SK6812MINI-E_3.2x2.8mm_P1.5mm_ReverseMount, B.Cu at (336.4, 139.2)
- added RGB82: SK6812MINI-E, my-keeb:LED_SK6812MINI-E_3.2x2.8mm_P1.5mm_ReverseMount, B.Cu at (355.5, 139.2)
- added RGB83: SK6812MINI-E, my-keeb:LED_SK6812MINI-E_3.2x2.8mm_P1.5mm_ReverseMount, B.Cu at (336.5, 101.5)
- added RGB84: SK6812MINI-E, my-keeb:LED_SK6812MINI-E_3.2x2.8mm_P1.5mm_ReverseMount, B.Cu at (355.6, 101.2)
- added RGB9: SK6812MINI-E, my-keeb:LED_SK6812MINI-E_3.2x2.8mm_P1.5mm_ReverseMount, B.Cu at (186.9, 44.2)
- added SW15: SW_Push, PCM_marbastlib-mx:SW_MX_1u, F.Cu at (253.6, 59.0)
- added SW94: SW_Push, PCM_marbastlib-mx:SW_MX_1u, F.Cu at (336.5, 97.2)
- added SW95: SW_Push, PCM_marbastlib-mx:SW_MX_1u, F.Cu at (355.6, 97.2)
- Capslock Key: renamed from SW44
- Enter Key: renamed from SW57
- Left Shift: renamed from SW58
- S3: footprint my-keeb:STAB_MX_P_2u -> my-keeb:STAB_MX_P_2.75u
- Tab Key: renamed from SW30
- ` ~ key: renamed from SW16
- moved H3 84.7 mm to (18.5, 99.0)
- moved H2 58.0 mm to (220.0, 34.5)
- moved D61 37.1 mm to (83.4, 106.5)
- moved D57 36.9 mm to (271.9, 86.0)
- moved SW77 31.1 mm to (146.4, 135.2)
- moved D77 29.7 mm to (142.7, 145.5)
- moved H1 26.2 mm to (41.0, 37.0)
- moved A1 22.9 mm to (313.9, 52.0)
- moved SW74 22.6 mm to (75.0, 135.2)
- moved SW79 20.8 mm to (217.9, 135.2)
- moved D74 20.5 mm to (70.5, 144.2)
- moved SW73 20.4 mm to (51.2, 135.2)
- moved SW92 20.0 mm to (355.5, 135.2)
- moved SW91 20.0 mm to (336.4, 135.2)
- moved SW93 20.0 mm to (317.4, 135.2)
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- renumbered SW2 to Escape
Connections:
- A1 pad 10: COL1 -> RGB_DATA
- A1 pad 36: unconnected-(A1-3V3-Pad36) -> 3V3
- D14 pad 2: Net-(D14-A) -> COL13
- SW14 pad 2: Net-(D14-A) -> COL13
Routing:
- net ROW5: track 487.2 -> 0.00 mm
- net ROW4: track 439.6 -> 0.00 mm, vias 1 -> 0
- net ROW2: track 424.7 -> 0.00 mm
- net ROW1: track 416.7 -> 0.00 mm
- net COL0: track 405.4 -> 0.00 mm
- net ROW0: track 392.0 -> 0.00 mm
- net ROW3: track 378.7 -> 0.00 mm
- net COL1: track 376.1 -> 0.00 mm
- net COL2: track 355.8 -> 0.00 mm
- net COL3: track 354.0 -> 0.00 mm
- net COL4: track 294.8 -> 0.00 mm
- net COL5: track 272.4 -> 0.00 mm
- net COL7: track 261.6 -> 0.00 mm
- net COL6: track 254.5 -> 0.00 mm
- net COL10: track 250.7 -> 0.00 mm
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- removed copper zone on B.Cu, net Net-(A1-GND-Pad13)
- removed copper zone on F.Cu, net Net-(A1-GND-Pad13)
Other:
- board size 360 x 170 mm -> 357 x 122 mm

Commit message: Add files via upload
Parts:
- removed H1, H2, H3, H4: MountingHole, MountingHole:MountingHole_3.2mm_M3
- removed MH1, MH2: MountingHole_3.048mm, MountingHole:MountingHole_3.048mm
- removed MH3, MH4: MountingHole_3.9878mm, MountingHole:MountingHole_3.9878mm
- added C1: 100nF, Capacitor_SMD:C_0603_1608Metric, F.Cu at (320.5, 84.5)
- added R1: 4.7k, Resistor_SMD:R_0603_1608Metric, F.Cu at (315.0, 84.5)
- added R2: 4.7k, Resistor_SMD:R_0603_1608Metric, F.Cu at (309.5, 84.5)
- added S8: MX_stab_6.25u, STAB_MX_P_6.25u, F.Cu at (146.5, 135.2)
- added U1: MCP23017x-x-SO, Package_SO:SOIC-28W_7.5x17.9mm_P1.27mm, F.Cu at (315.0, 98.0)
- RGB1, RGB10, RGB11, RGB12, RGB13, RGB14, RGB15, RGB16, RGB17, RGB18, RGB19, RGB2, RGB20, RGB21, RGB22, RGB23, RGB24, RGB25, RGB26, RGB27, RGB28, RGB29, RGB3, RGB30, RGB31, RGB32, RGB33, RGB35, RGB36, RGB37, RGB38, RGB39, RGB4, RGB40, RGB41, RGB42, RGB43, RGB44, RGB45, RGB46, RGB47, RGB48, RGB49, RGB5, RGB50, RGB51, RGB52, RGB53, RGB54, RGB55, RGB56, RGB57, RGB58, RGB59, RGB6, RGB60, RGB61, RGB62, RGB63, RGB64, RGB65, RGB66, RGB67, RGB68, RGB69, RGB7, RGB70, RGB71, RGB72, RGB73, RGB74, RGB75, RGB76, RGB77, RGB78, RGB79, RGB8, RGB80, RGB81, RGB82, RGB83, RGB84, RGB9: footprint my-keeb:LED_SK6812MINI-E_3.2x2.8mm_P1.5mm_ReverseMount -> LED_SMD:LED_SK6812MINI-E_3.2x2.8mm_P1.5mm_ReverseMount
- S3: footprint my-keeb:STAB_MX_P_2.75u -> my-keeb:STAB_MX_P_2u
- S7: footprint my-keeb:STAB_MX_P_2u -> STAB_MX_P_2u
- SW16: renamed from ` ~ key
- SW30: renamed from Tab Key
- SW44: renamed from Capslock Key
- SW57: renamed from Enter Key
- SW58: renamed from Left Shift
- moved D11 43.1 mm to (234.6, 49.0)
- moved D12 43.1 mm to (253.6, 49.0)
- moved D14 43.1 mm to (291.7, 49.0)
- moved D13 43.1 mm to (272.6, 49.0)
- moved D7 33.6 mm to (148.8, 49.0)
- moved D9 33.6 mm to (186.9, 49.0)
- moved D10 33.6 mm to (206.0, 49.0)
- moved D8 33.6 mm to (167.9, 49.0)
- moved D29 27.7 mm to (282.2, 68.0)
- moved D15 25.2 mm to (253.6, 68.0)
- moved D3 24.1 mm to (63.1, 49.0)
- moved D4 24.1 mm to (82.2, 49.0)
- moved D5 24.0 mm to (101.2, 49.0)
- moved D6 24.0 mm to (120.2, 49.0)
- moved D57 21.6 mm to (279.8, 106.2)
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- renumbered Escape to SW2
Connections:
- net COL0 renamed /COL0
- net COL1 renamed /COL1
- net COL10 renamed /COL10
- net COL11 renamed /COL11
- net COL12 renamed /COL12
- net COL14 renamed /COL14
- net COL15 renamed /COL15
- net COL16 renamed /COL16
- net COL2 renamed /COL2
- net COL3 renamed /COL3
- net COL4 renamed /COL4
- net COL5 renamed /COL5
- net COL6 renamed /COL6
- net COL7 renamed /COL7
- net COL8 renamed /COL8
- net COL9 renamed /COL9
- net KEY94 renamed /KEY94
- net KEY95 renamed /KEY95
- net ROW0 renamed /ROW0
- net ROW1 renamed /ROW1
- net ROW2 renamed /ROW2
- net ROW3 renamed /ROW3
- net ROW4 renamed /ROW4
- net ROW5 renamed /ROW5
- A1 pad 13: Net-(A1-GND-Pad13) -> unconnected-(A1-GND-Pad13)_12
- A1 pad 18: Net-(A1-GND-Pad13) -> unconnected-(A1-GND-Pad13)_10
- A1 pad 23: Net-(A1-GND-Pad13) -> unconnected-(A1-GND-Pad13)_7
- A1 pad 25: COL13 -> /COL13
- A1 pad 28: Net-(A1-GND-Pad13) -> unconnected-(A1-GND-Pad13)
- A1 pad 3: Net-(A1-GND-Pad13) -> unconnected-(A1-GND-Pad13)_11
- A1 pad 31: unconnected-(A1-GPIO26_ADC0-Pad31) -> I2C_SDA
- A1 pad 32: unconnected-(A1-GPIO27_ADC1-Pad32) -> I2C_SCL
- A1 pad 34: unconnected-(A1-GPIO28_ADC2-Pad34) -> MCP23017_INT
- A1 pad 38: Net-(A1-GND-Pad13) -> unconnected-(A1-GND-Pad13)_5
- A1 pad 8: Net-(A1-GND-Pad13) -> unconnected-(A1-GND-Pad13)_6
- D14 pad 2: COL13 -> Net-(D14-A)
- ENC1 pad A: (no net) -> ENC1_A
- ENC1 pad B: (no net) -> ENC1_B
- ENC1 pad C: (no net) -> 3V3
- ENC1 pad S1: (no net) -> ENC1_SW
- ENC1 pad S2: (no net) -> 3V3
- ENC2 pad A: (no net) -> ENC2_A
- ENC2 pad B: (no net) -> ENC2_B
- ENC2 pad C: (no net) -> 3V3
- ENC2 pad S1: (no net) -> ENC2_SW
- ENC2 pad S2: (no net) -> 3V3
- RGB24 pad 3: GND -> 3V3
- RGB3 pad 1: GND -> 3V3
- RGB41 pad 1: GND -> 3V3
- RGB43 pad 1: GND -> 3V3
- RGB44 pad 1: GND -> 3V3
- RGB46 pad 1: GND -> 3V3
- RGB5 pad 1: GND -> 3V3
- RGB57 pad 4: RGB_83 -> RGB_57
- RGB58 pad 2: RGB_57 -> RGB_84
- RGB60 pad 1: GND -> 3V3
- RGB61 pad 1: GND -> 3V3
- RGB62 pad 1: GND -> 3V3
- RGB63 pad 1: GND -> 3V3
- RGB64 pad 1: GND -> 3V3
- RGB65 pad 1: GND -> 3V3
- RGB66 pad 1: GND -> 3V3
- RGB71 pad 1: GND -> 3V3
- RGB72 pad 1: GND -> 3V3
- RGB73 pad 1: GND -> 3V3
- RGB74 pad 1: GND -> 3V3
- RGB75 pad 1: GND -> 3V3
- RGB76 pad 1: GND -> 3V3
- RGB77 pad 1: GND -> 3V3
- RGB78 pad 1: GND -> 3V3
- RGB79 pad 1: GND -> 3V3
- RGB80 pad 1: GND -> 3V3
- RGB81 pad 1: GND -> 3V3
- RGB82 pad 1: GND -> 3V3
- RGB83 pad 1: GND -> 3V3
- RGB83 pad 2: RGB_83 -> RGB_57
- RGB83 pad 4: RGB_84 -> RGB_83
- RGB84 pad 1: GND -> 3V3
- RGB84 pad 2: RGB_84 -> RGB_83
- RGB84 pad 4: RGB_57 -> RGB_84
- SW14 pad 2: COL13 -> Net-(D14-A)
- SW15 pad 1: COL13 -> /COL13
- SW29 pad 1: COL13 -> /COL13
- SW43 pad 1: COL13 -> /COL13
- SW57 pad 1: COL13 -> /COL13
- SW71 pad 1: COL13 -> /COL13
- SW82 pad 1: COL13 -> /COL13
Routing:
- net 3V3: track 0.00 -> 3149.7 mm, vias 0 -> 6
- net /ROW5: track 0.00 -> 457.9 mm
- net /ROW3: track 0.00 -> 416.7 mm, vias 0 -> 1
- net /ROW2: track 0.00 -> 406.1 mm
- net /ROW4: track 0.00 -> 402.5 mm, vias 0 -> 1
- net /COL0: track 0.00 -> 401.0 mm
- net /COL2: track 0.00 -> 400.3 mm, vias 0 -> 2
- net /ROW1: track 0.00 -> 387.0 mm, vias 0 -> 1
- net RGB_84: track 0.00 -> 342.1 mm, vias 0 -> 4
- net /COL3: track 0.00 -> 340.6 mm
- net /ROW0: track 0.00 -> 339.1 mm
- net RGB_29: track 0.00 -> 334.5 mm, vias 0 -> 2
- net RGB_70: track 0.00 -> 319.1 mm, vias 0 -> 2
- net /COL4: track 0.00 -> 317.9 mm, vias 0 -> 3
- net RGB_45: track 0.00 -> 309.5 mm, vias 0 -> 2
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Other:
- board size 357 x 122 mm -> 361.7 x 122 mm
