File: my-keeb.kicad_pcb (KiCad board)
At the start: 2 copper layers, 355.7 x 122 mm, 264 parts, among them SW10 SW_Push, SW11 SW_Push, SW12 SW_Push, SW13 SW_Push, SW14 SW_Push, SW15 SW_Push, SW16 SW_Push, SW17 SW_Push, SW18 SW_Push, SW19 SW_Push, SW2 SW_Push, SW20 SW_Push, SW21 SW_Push, SW22 SW_Push, SW23 SW_Push, SW24 SW_Push, SW25 SW_Push, SW26 SW_Push, SW27 SW_Push, SW29 SW_Push, SW3 SW_Push, SW30 SW_Push, SW31 SW_Push, SW32 SW_Push, SW33 SW_Push, SW34 SW_Push, SW35 SW_Push, SW36 SW_Push, SW37 SW_Push, SW38 SW_Push, SW39 SW_Push, SW4 SW_Push, SW40 SW_Push, SW41 SW_Push, SW42 SW_Push, SW43 SW_Push, SW44 SW_Push, SW45 SW_Push, SW46 SW_Push, SW47 SW_Push, SW48 SW_Push, SW49 SW_Push, SW5 SW_Push, SW50 SW_Push, SW51 SW_Push, SW52 SW_Push, SW53 SW_Push, SW54 SW_Push, SW55 SW_Push, SW57 SW_Push, SW58 SW_Push, SW6 SW_Push, SW60 SW_Push, SW61 SW_Push, SW62 SW_Push, SW63 SW_Push, SW64 SW_Push, SW65 SW_Push, SW66 SW_Push, SW67 SW_Push, SW68 SW_Push, SW69 SW_Push, SW7 SW_Push, SW71 SW_Push, SW72 SW_Push, SW73 SW_Push, SW74 SW_Push, SW77 SW_Push, SW79 SW_Push, SW8 SW_Push, SW80 SW_Push, SW81 SW_Push, SW82 SW_Push, SW86 SW_Push, SW87 SW_Push, SW88 SW_Push, SW89 SW_Push, SW9 SW_Push, SW90 SW_Push, SW91 SW_Push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

Commit message: Added mising connection for COL0
Connections:
- U1 pad 27: unconnected-(U1-GPA6-Pad27) -> /COL1
Routing:
- net /COL1: track 126.5 -> 403.2 mm, vias 0 -> 1
Changed lines of the file:
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@@
 			(layers "F.Cu" "F.Mask" "F.Paste")
 			(roundrect_rratio 0.25)
-			(net "unconnected-(U1-GPA6-Pad27)")
+			(net "/COL1")
 			(pinfunction "GPA6_27")
-			(pintype "bidirectional+no_connect")
+			(pintype "bidirectional")
 		)
 		(pad "28" smd roundrect
@@
 	)
 	(segment
+		(start 289 93.25)
+		(end 284 88.25)
+		(width 0.2)
+		(layer "F.Cu")
+		(net "/COL1")
+	)
+	(segment
 		(start 44.31 75.56)
 		(end 36.75 68)
@@
 	)
 	(segment
+		(start 318.515 91.015)
+		(end 315.25 87.75)
+		(width 0.2)
+		(layer "F.Cu")
+		(net "/COL1")
+	)
+	(segment
 		(start 38.613655 56.51)
 		(end 40.24 56.51)
@@
 	)
 	(segment
+		(start 319.65 91.015)
+		(end 318.515 91.015)
+		(width 0.2)
+		(layer "F.Cu")
+		(net "/COL1")
+	)
+	(segment
+		(start 293.5 93.25)
+		(end 289 93.25)
+		(width 0.2)
+		(layer "F.Cu")
+		(net "/COL1")
+	)
+	(segment
 		(start 40.24 54.883655)
 		(end 40.24 56.51)
@@
 	)
 	(segment
+		(start 299 87.75)
+		(end 293.5 93.25)
+		(width 0.2)
+		(layer "F.Cu")
+		(net "/COL1")
+	)
+	(segment
 		(start 36.75 68)
 		(end 36.75 58.373655)
@@
 	)
 	(segment
+		(start 284 88.25)
+		(end 282.75 88.25)
+		(width 0.2)
+		(layer "F.Cu")
+		(net "/COL1")
+	)
+	(segment
 		(start 44.31 75.56)
 		(end 44.31 91.56)
@@
 	)
 	(segment
+		(start 315.25 87.75)
+		(end 299 87.75)
+		(width 0.2)
+		(layer "F.Cu")
+		(net "/COL1")
+	)
+	(via
+		(at 282.75 88.25)
+		(size 0.6)
+		(drill 0.3)
+		(layers "F.Cu" "B.Cu")
+		(net "/COL1")
+	)
+	(segment
+		(start 59.38 89.75)
+		(end 54.52 94.61)
+		(width 0.2)
+		(layer "B.Cu")
+		(net "/COL1")
+	)
+	(segment
+		(start 282.75 88.25)
+		(end 274.75 88.25)
+		(width 0.2)
+		(layer "B.Cu")
+		(net "/COL1")
+	)
+	(segment
+		(start 252.75 89.75)
+		(end 59.38 89.75)
+		(width 0.2)
+		(layer "B.Cu")
+		(net "/COL1")
+	)
+	(segment
+		(start 274.75 88.25)
+		(end 269.25 93.75)
+		(width 0.2)
+		(layer "B.Cu")
+		(net "/COL1")
+	)
+	(segment
+		(start 269.25 93.75)
+		(end 256.75 93.75)
+		(width 0.2)
+		(layer "B.Cu")
+		(net "/COL1")
+	)
+	(segment
+		(start 256.75 93.75)
+		(end 252.75 89.75)
+		(width 0.2)
+		(layer "B.Cu")
+		(net "/COL1")
+	)
+	(segment
 		(start 46.59 53.97)
 		(end 51.67 59.05)
@@
 	)
 	(segment
-		(start 319.65 94.825)
-		(end 319.075 94.825)
+		(start 319.075 94.825)
+		(end 319.65 94.825)
 		(width 0.2)
 		(layer "F.Cu")
@@
 	)
 	(segment
-		(start 319.075 94.825)
-		(end 313.25 89)
+		(start 314.025 89.775)
+		(end 319.075 94.825)
 		(width 0.2)
 		(layer "F.Cu")
@@
 	)
 	(segment
-		(start 313.25 89)
-		(end 313.25 87.7)
+		(start 314.025 88.475)
+		(end 314.025 89.775)
 		(width 0.2)
 		(layer "F.Cu")
@@
 	)
 	(via
-		(at 313.25 87.7)
+		(at 314.025 88.475)
 		(size 0.6)
 		(drill 0.3)
@@
 	)
 	(segment
-		(start 319.1 42.1)
-		(end 319.1 32.65)
+		(start 319.935 31.815)
+		(end 323.185 31.815)
 		(width 0.2)
 		(layer "B.Cu")
@@
 	)
 	(segment
-		(start 313.25 84.25)
-		(end 313.25 87.7)
+		(start 306.725 77.725)
+		(end 306.725 68.928578)
 		(width 0.2)
 		(layer "B.Cu")
@@
 	)
 	(segment
-		(start 347.6 31.1)
-		(end 352 35.5)
+		(start 319.1 42.1)
+		(end 319.1 32.65)
 		(width 0.2)
 		(layer "B.Cu")
@@
 	)
 	(segment
-		(start 313.25 84.25)
-		(end 306.725 77.725)
+		(start 314.025 88.475)
+		(end 313.25 87.7)
 		(width 0.2)
 		(layer "B.Cu")
@@
 	)
 	(segment
-		(start 323.9 31.1)
-		(end 347.6 31.1)
+		(start 313.25 87.7)
+		(end 313.25 84.25)
 		(width 0.2)
 		(layer "B.Cu")
@@
 	)
 	(segment
-		(start 323.185 31.815)
-		(end 323.9 31.1)
+		(start 306.725 68.928578)
+		(end 316.903578 58.75)
 		(width 0.2)
 		(layer "B.Cu")
@@
 	)
 	(segment
-		(start 319.935 31.815)
-		(end 323.185 31.815)
+		(start 320.75 58.75)
+		(end 320.75 43.75)
 		(width 0.2)
 		(layer "B.Cu")
@@
 	)
 	(segment
-		(start 319.1 32.65)
-		(end 319.935 31.815)
+		(start 323.185 31.815)
+		(end 323.9 31.1)
 		(width 0.2)
 		(layer "B.Cu")
@@
 	)
 	(segment
-		(start 316.903578 58.75)
-		(end 320.75 58.75)
+		(start 323.9 31.1)
+		(end 347.6 31.1)
 		(width 0.2)
 		(layer "B.Cu")
@@
 	)
 	(segment
-		(start 306.725 77.725)
-		(end 306.725 68.928578)
+		(start 319.1 32.65)
+		(end 319.935 31.815)
 		(width 0.2)
 		(layer "B.Cu")
@@
 	)
 	(segment
-		(start 320.75 58.75)
-		(end 320.75 43.75)
+		(start 313.25 84.25)
+		(end 306.725 77.725)
 		(width 0.2)
 		(layer "B.Cu")
@@
 	)
 	(segment
-		(start 306.725 68.928578)
-		(end 316.903578 58.75)
+		(start 347.6 31.1)
+		(end 352 35.5)
+		(width 0.2)
+		(layer "B.Cu")
+		(net "ENC2_A")
+	)
+	(segment
+		(start 316.903578 58.75)
+		(end 320.75 58.75)
 		(width 0.2)
 		(layer "B.Cu")

Commit message: Add files via upload
Parts:
- removed C1: 100nF, Capacitor_SMD:C_0603_1608Metric
- removed R1, R2: 4.7k, Resistor_SMD:R_0603_1608Metric
- removed U1: MCP23017x-x-SO, Package_SO:SOIC-28W_7.5x17.9mm_P1.27mm
- added D1: 1N4148, Diode_THT:D_DO-35_SOD27_P7.62mm_Horizontal, F.Cu at (355.7, 46.8)
- added D28: 1N4148, Diode_THT:D_DO-35_SOD27_P7.62mm_Horizontal, F.Cu at (333.5, 46.8)
- ENC1: value EC11 -> MUTE_MIC
- ENC2: value EC11 -> MUTE_SOUND
- SW10: value SW_Push -> F8
- SW11: value SW_Push -> F9
- SW12: value SW_Push -> F10
- SW13: value SW_Push -> F11
- SW14: value SW_Push -> F12
- SW15: value SW_Push -> =
- SW16: value SW_Push -> `
- SW17: value SW_Push -> 1
- SW18: value SW_Push -> 2
- SW19: value SW_Push -> 3
- SW2: value SW_Push -> ESC
- SW20: value SW_Push -> 4
- SW21: value SW_Push -> 5
- SW22: value SW_Push -> 6
- SW23: value SW_Push -> 7
- SW24: value SW_Push -> 8
- SW25: value SW_Push -> 9
- SW26: value SW_Push -> 0
- SW27: value SW_Push -> -
- SW29: value SW_Push -> BACKSPACE
- SW3: value SW_Push -> F1
- SW30: value SW_Push -> TAB
- SW31: value SW_Push -> Q
- SW32: value SW_Push -> W
- SW33: value SW_Push -> E
- SW34: value SW_Push -> R
- SW35: value SW_Push -> T
- SW36: value SW_Push -> Y
- SW37: value SW_Push -> U
- SW38: value SW_Push -> I
- SW39: value SW_Push -> O
- SW4: value SW_Push -> F2
- SW40: value SW_Push -> P
- SW41: value SW_Push -> [
- SW42: value SW_Push -> ]
- SW43: value SW_Push -> \
- SW44: value SW_Push -> CAPSLOCK
- SW45: value SW_Push -> A
- SW46: value SW_Push -> S
- SW47: value SW_Push -> D
- SW48: value SW_Push -> F
- SW49: value SW_Push -> G
- SW5: value SW_Push -> F3
- SW50: value SW_Push -> H
- SW51: value SW_Push -> J
- SW52: value SW_Push -> K
- SW53: value SW_Push -> L
- SW54: value SW_Push -> ;
- SW55: value SW_Push -> '
- SW57: value SW_Push -> ENTER
- SW58: value SW_Push -> LEFT_SHIFT
- SW6: value SW_Push -> F4
- SW60: value SW_Push -> Z
- SW61: value SW_Push -> X
- SW62: value SW_Push -> C
- SW63: value SW_Push -> V
- SW64: value SW_Push -> B
- SW65: value SW_Push -> N
- SW66: value SW_Push -> M
- SW67: value SW_Push -> ,
- SW68: value SW_Push -> .
- SW69: value SW_Push -> /
- SW7: value SW_Push -> F5
- SW71: value SW_Push -> RIGHT_SHIFT
- SW72, SW82: value SW_Push -> CTRL
- SW73, SW80: value SW_Push -> WINDOWS_KEY
- SW74, SW79: value SW_Push -> ALT
- SW77: value SW_Push -> SPACEBAR
- SW8: value SW_Push -> F6
- SW81: value SW_Push -> FN
- SW86: value SW_Push -> PRT SC
- SW87: value SW_Push -> WINDOWS_KEY_PLUS_PERIOD
- SW88: value SW_Push -> INS
- SW89: value SW_Push -> PG_UP
- SW9: value SW_Push -> F7
- SW90: value SW_Push -> UP_ARROW
- SW91: value SW_Push -> DOWN_ARROW
- SW92: value SW_Push -> RIGHT_ARROW
- SW93: value SW_Push -> LEFT_ARROW
- SW94: value SW_Push -> DEL
- SW95: value SW_Push -> PG_DN
Connections:
- A1 pad 10: RGB_DATA -> /COL1
- A1 pad 13: unconnected-(A1-GND-Pad13)_12 -> 3V3
- A1 pad 18: unconnected-(A1-GND-Pad13)_10 -> 3V3
- A1 pad 23: unconnected-(A1-GND-Pad13)_7 -> 3V3
- A1 pad 27: /COL15 -> ENC2_A
- A1 pad 28: unconnected-(A1-GND-Pad13) -> 3V3
- A1 pad 29: /COL16 -> ENC2_B
- A1 pad 3: unconnected-(A1-GND-Pad13)_11 -> 3V3
- A1 pad 31: I2C_SDA -> RGB_DATA
- A1 pad 32: I2C_SCL -> ENC1_A
- A1 pad 34: MCP23017_INT -> ENC1_B
- A1 pad 38: unconnected-(A1-GND-Pad13)_5 -> 3V3
- A1 pad 8: unconnected-(A1-GND-Pad13)_6 -> 3V3
- D87 pad 1: /ROW1 -> /ROW4
- D89 pad 1: /ROW2 -> /ROW4
- ENC1 pad S1: ENC1_SW -> Net-(D28-A)
- ENC1 pad S2: 3V3 -> /COL14
- ENC2 pad S1: ENC2_SW -> Net-(D1-A)
- ENC2 pad S2: 3V3 -> /COL14
- SW86 pad 1: /COL15 -> /COL12
- SW87 pad 1: /COL16 -> /COL1
- SW88 pad 1: /COL15 -> /COL14
- SW89 pad 1: /COL16 -> /COL12
- SW90 pad 1: /COL15 -> /COL14
- SW91 pad 1: /COL15 -> /COL3
- SW92 pad 1: /COL16 -> /COL4
- SW95 pad 1: /COL15 -> /COL12
Routing:
- net /COL3: track 343.2 -> 628.2 mm
- net /COL4: track 333.1 -> 609.7 mm, vias 0 -> 2
- net /COL14: track 109.4 -> 326.5 mm
- net /COL15: track 157.1 -> 0.00 mm
- net /ROW4: track 396.9 -> 541.5 mm, vias 2 -> 3
- net /COL16: track 135.6 -> 0.00 mm
- net /COL1: track 403.2 -> 511.3 mm, vias 1 -> 3
- net ENC1_SW: track 89.9 -> 0.00 mm, vias 1 -> 0
- net ENC2_SW: track 88.9 -> 0.00 mm, vias 5 -> 0
- net /COL12: track 249.2 -> 329.1 mm, vias 0 -> 2
- net ENC2_B: track 117.3 -> 41.0 mm, vias 1 -> 0
- net I2C_SCL: track 74.2 -> 0.00 mm, vias 3 -> 0
- net MCP23017_INT: track 68.2 -> 0.00 mm, vias 4 -> 0
- net I2C_SDA: track 64.9 -> 0.00 mm, vias 3 -> 0
- net ENC1_B: track 77.2 -> 21.1 mm
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
Commit message: Add files via upload
Parts:
- ENC1: value MUTE_MIC -> EC11
- ENC2: value MUTE_SOUND -> EC11
- S8: footprint STAB_MX_P_6.25u -> my-keeb:STAB_MX_P_6.25u
- SW10: value F8 -> SW_Push
- SW11: value F9 -> SW_Push
- SW12: value F10 -> SW_Push
- SW13: value F11 -> SW_Push
- SW14: value F12 -> SW_Push
- SW15: value = -> SW_Push
- SW16: value ` -> SW_Push
- SW17: value 1 -> SW_Push
- SW18: value 2 -> SW_Push
- SW19: value 3 -> SW_Push
- SW2: value ESC -> SW_Push
- SW20: value 4 -> SW_Push
- SW21: value 5 -> SW_Push
- SW22: value 6 -> SW_Push
- SW23: value 7 -> SW_Push
- SW24: value 8 -> SW_Push
- SW25: value 9 -> SW_Push
- SW26: value 0 -> SW_Push
- SW27: value - -> SW_Push
- SW29: value BACKSPACE -> SW_Push
- SW3: value F1 -> SW_Push
- SW30: value TAB -> SW_Push
- SW31: value Q -> SW_Push
- SW32: value W -> SW_Push
- SW33: value E -> SW_Push
- SW34: value R -> SW_Push
- SW35: value T -> SW_Push
- SW36: value Y -> SW_Push
- SW37: value U -> SW_Push
- SW38: value I -> SW_Push
- SW39: value O -> SW_Push
- SW4: value F2 -> SW_Push
- SW40: value P -> SW_Push
- SW41: value [ -> SW_Push
- SW42: value ] -> SW_Push
- SW43: value \ -> SW_Push
- SW44: value CAPSLOCK -> SW_Push
- SW45: value A -> SW_Push
- SW46: value S -> SW_Push
- SW47: value D -> SW_Push
- SW48: value F -> SW_Push
- SW49: value G -> SW_Push
- SW5: value F3 -> SW_Push
- SW50: value H -> SW_Push
- SW51: value J -> SW_Push
- SW52: value K -> SW_Push
- SW53: value L -> SW_Push
- SW54: value ; -> SW_Push
- SW55: value ' -> SW_Push
- SW57: value ENTER -> SW_Push
- SW58: value LEFT_SHIFT -> SW_Push
- SW6: value F4 -> SW_Push
- SW60: value Z -> SW_Push
- SW61: value X -> SW_Push
- SW62: value C -> SW_Push
- SW63: value V -> SW_Push
- SW64: value B -> SW_Push
- SW65: value N -> SW_Push
- SW66: value M -> SW_Push
- SW67: value , -> SW_Push
- SW68: value . -> SW_Push
- SW69: value / -> SW_Push
- SW7: value F5 -> SW_Push
- SW71: value RIGHT_SHIFT -> SW_Push
- SW72, SW82: value CTRL -> SW_Push
- SW73, SW80: value WINDOWS_KEY -> SW_Push
- SW74, SW79: value ALT -> SW_Push
- SW77: value SPACEBAR -> SW_Push
- SW8: value F6 -> SW_Push
- SW81: value FN -> SW_Push
- SW86: value PRT SC -> SW_Push
- SW87: value WINDOWS_KEY_PLUS_PERIOD -> SW_Push
- SW88: value INS -> SW_Push
- SW89: value PG_UP -> SW_Push
- SW9: value F7 -> SW_Push
- SW90: value UP_ARROW -> SW_Push
- SW91: value DOWN_ARROW -> SW_Push
- SW92: value RIGHT_ARROW -> SW_Push
- SW93: value LEFT_ARROW -> SW_Push
- SW94: value DEL -> SW_Push
- SW95: value PG_DN -> SW_Push
- moved D91 6.18 mm to (342.6, 144.2)
- moved D73 0.31 mm to (51.4, 144.5)
Connections:
- net RGB_1 renamed RGB_D1
- net RGB_10 renamed RGB_D10
- net RGB_11 renamed RGB_D11
- net RGB_12 renamed RGB_D12
- net RGB_13 renamed RGB_D13
- net RGB_14 renamed RGB_D14
- net RGB_15 renamed RGB_D15
- net RGB_16 renamed RGB_D16
- net RGB_17 renamed RGB_D17
- net RGB_18 renamed RGB_D18
- net RGB_19 renamed RGB_D19
- net RGB_2 renamed RGB_D2
- net RGB_20 renamed RGB_D20
- net RGB_21 renamed RGB_D21
- net RGB_22 renamed RGB_D22
- net RGB_23 renamed RGB_D23
- net RGB_24 renamed RGB_D24
- net RGB_25 renamed RGB_D25
- net RGB_26 renamed RGB_D26
- net RGB_27 renamed RGB_D27
- net RGB_28 renamed RGB_D28
- net RGB_29 renamed RGB_D29
- net RGB_3 renamed RGB_D3
- net RGB_30 renamed RGB_D30
- net RGB_31 renamed RGB_D31
- net RGB_32 renamed RGB_D32
- net RGB_33 renamed RGB_D33
- net RGB_34 renamed RGB_D34
- net RGB_35 renamed RGB_D35
- net RGB_36 renamed RGB_D36
- net RGB_37 renamed RGB_D37
- net RGB_38 renamed RGB_D38
- net RGB_39 renamed RGB_D39
- net RGB_4 renamed RGB_D4
- net RGB_40 renamed RGB_D40
- net RGB_41 renamed RGB_D41
- net RGB_42 renamed RGB_D42
- net RGB_43 renamed RGB_D43
- net RGB_44 renamed RGB_D44
- net RGB_45 renamed RGB_D45
- net RGB_46 renamed RGB_D46
- net RGB_47 renamed RGB_D47
- net RGB_48 renamed RGB_D48
- net RGB_49 renamed RGB_D49
- net RGB_5 renamed RGB_D5
- net RGB_50 renamed RGB_D50
- net RGB_51 renamed RGB_D51
- net RGB_52 renamed RGB_D52
- net RGB_53 renamed RGB_D53
- net RGB_54 renamed RGB_D54
- net RGB_55 renamed RGB_D55
- net RGB_56 renamed RGB_D56
- net RGB_58 renamed RGB_D58
- net RGB_59 renamed RGB_D59
- net RGB_6 renamed RGB_D6
- net RGB_60 renamed RGB_D60
- net RGB_61 renamed RGB_D61
- net RGB_62 renamed RGB_D62
- net RGB_63 renamed RGB_D63
- net RGB_64 renamed RGB_D64
- net RGB_65 renamed RGB_D65
- net RGB_66 renamed RGB_D66
- net RGB_67 renamed RGB_D67
- net RGB_68 renamed RGB_D68
- net RGB_69 renamed RGB_D69
- net RGB_7 renamed RGB_D7
- net RGB_70 renamed RGB_D70
- net RGB_71 renamed RGB_D71
- net RGB_72 renamed RGB_D72
- net RGB_73 renamed RGB_D73
- net RGB_74 renamed RGB_D74
- net RGB_75 renamed RGB_D75
- net RGB_76 renamed RGB_D76
- net RGB_77 renamed RGB_D77
- net RGB_78 renamed RGB_D78
- net RGB_79 renamed RGB_D79
- net RGB_8 renamed RGB_D8
- net RGB_80 renamed RGB_D80
- net RGB_81 renamed RGB_D81
- net RGB_83 renamed RGB_D83
- net RGB_9 renamed RGB_D9
- A1 pad 13: 3V3 -> GND
- A1 pad 18: 3V3 -> GND
- A1 pad 23: 3V3 -> GND
- A1 pad 28: 3V3 -> GND
- A1 pad 3: 3V3 -> GND
- A1 pad 36: 3V3 -> unconnected-(A1-3V3-Pad36)
- A1 pad 38: 3V3 -> GND
- A1 pad 40: unconnected-(A1-VBUS-Pad40)_1 -> +5V
- A1 pad 8: 3V3 -> GND
- ENC1 pad C: 3V3 -> GND
- ENC2 pad C: 3V3 -> GND
- RGB1 pad 1: 3V3 -> GND
- RGB1 pad 3: 3V3 -> +5V
- RGB10 pad 1: 3V3 -> GND
- RGB10 pad 3: 3V3 -> +5V
- RGB11 pad 1: 3V3 -> GND
- RGB11 pad 3: 3V3 -> +5V
- RGB12 pad 1: 3V3 -> GND
- RGB12 pad 3: 3V3 -> +5V
- RGB13 pad 1: 3V3 -> GND
- RGB13 pad 3: 3V3 -> +5V
- RGB14 pad 1: 3V3 -> GND
- RGB14 pad 3: 3V3 -> +5V
- RGB15 pad 1: 3V3 -> GND
- RGB15 pad 3: 3V3 -> +5V
- RGB16 pad 1: 3V3 -> GND
- RGB16 pad 3: 3V3 -> +5V
- RGB17 pad 1: 3V3 -> GND
- RGB17 pad 3: 3V3 -> +5V
- RGB18 pad 1: 3V3 -> GND
- RGB18 pad 3: 3V3 -> +5V
- RGB19 pad 1: 3V3 -> GND
- RGB19 pad 3: 3V3 -> +5V
- RGB2 pad 1: 3V3 -> GND
- RGB2 pad 3: 3V3 -> +5V
- RGB20 pad 1: 3V3 -> GND
- RGB20 pad 3: 3V3 -> +5V
- RGB21 pad 1: 3V3 -> GND
- RGB21 pad 3: 3V3 -> +5V
- RGB22 pad 1: 3V3 -> GND
- RGB22 pad 3: 3V3 -> +5V
- RGB23 pad 1: 3V3 -> GND
- RGB23 pad 3: 3V3 -> +5V
- RGB24 pad 1: 3V3 -> GND
- RGB24 pad 3: 3V3 -> +5V
- RGB25 pad 1: 3V3 -> GND
- RGB25 pad 3: 3V3 -> +5V
- RGB26 pad 1: 3V3 -> GND
- RGB26 pad 3: 3V3 -> +5V
- RGB27 pad 1: 3V3 -> GND
- RGB27 pad 3: 3V3 -> +5V
- RGB28 pad 1: 3V3 -> GND
- RGB28 pad 3: 3V3 -> +5V
- RGB29 pad 1: 3V3 -> GND
- RGB29 pad 3: 3V3 -> +5V
- RGB3 pad 1: 3V3 -> GND
- RGB3 pad 3: 3V3 -> +5V
- RGB30 pad 1: 3V3 -> GND
- RGB30 pad 3: 3V3 -> +5V
- RGB31 pad 1: 3V3 -> GND
- RGB31 pad 3: 3V3 -> +5V
- RGB32 pad 1: 3V3 -> GND
- RGB32 pad 3: 3V3 -> +5V
- RGB33 pad 1: 3V3 -> GND
- RGB33 pad 3: 3V3 -> +5V
- RGB34 pad 1: 3V3 -> GND
- RGB34 pad 3: 3V3 -> +5V
- RGB35 pad 1: 3V3 -> GND
- RGB35 pad 3: 3V3 -> +5V
- RGB36 pad 1: 3V3 -> GND
- RGB36 pad 3: 3V3 -> +5V
- RGB37 pad 1: 3V3 -> GND
- RGB37 pad 3: 3V3 -> +5V
- RGB38 pad 1: 3V3 -> GND
- RGB38 pad 3: 3V3 -> +5V
- RGB39 pad 1: 3V3 -> GND
- RGB39 pad 3: 3V3 -> +5V
- RGB4 pad 1: 3V3 -> GND
- RGB4 pad 3: 3V3 -> +5V
- RGB40 pad 1: 3V3 -> GND
- RGB40 pad 3: 3V3 -> +5V
- RGB41 pad 1: 3V3 -> GND
- RGB41 pad 3: 3V3 -> +5V
- RGB42 pad 1: 3V3 -> GND
- RGB42 pad 3: 3V3 -> +5V
- RGB43 pad 1: 3V3 -> GND
- RGB43 pad 3: 3V3 -> +5V
- RGB44 pad 1: 3V3 -> GND
- RGB44 pad 3: 3V3 -> +5V
- RGB45 pad 1: 3V3 -> GND
- RGB45 pad 3: 3V3 -> +5V
- RGB46 pad 1: 3V3 -> GND
- RGB46 pad 3: 3V3 -> +5V
- RGB47 pad 1: 3V3 -> GND
- RGB47 pad 3: 3V3 -> +5V
- RGB48 pad 1: 3V3 -> GND
- RGB48 pad 3: 3V3 -> +5V
- RGB49 pad 1: 3V3 -> GND
- RGB49 pad 3: 3V3 -> +5V
- RGB5 pad 1: 3V3 -> GND
- RGB5 pad 3: 3V3 -> +5V
- RGB50 pad 1: 3V3 -> GND
- RGB50 pad 3: 3V3 -> +5V
- RGB51 pad 1: 3V3 -> GND
- RGB51 pad 3: 3V3 -> +5V
- RGB52 pad 1: 3V3 -> GND
- RGB52 pad 3: 3V3 -> +5V
- RGB53 pad 1: 3V3 -> GND
- RGB53 pad 3: 3V3 -> +5V
- RGB54 pad 1: 3V3 -> GND
- RGB54 pad 3: 3V3 -> +5V
- RGB55 pad 1: 3V3 -> GND
- RGB55 pad 3: 3V3 -> +5V
- RGB56 pad 1: 3V3 -> GND
- RGB56 pad 3: 3V3 -> +5V
- RGB57 pad 1: 3V3 -> GND
- RGB57 pad 3: 3V3 -> +5V
- RGB57 pad 4: RGB_57 -> RGB_D57
- RGB58 pad 1: 3V3 -> GND
- RGB58 pad 2: RGB_84 -> RGB_D57
- RGB58 pad 3: 3V3 -> +5V
- RGB59 pad 1: 3V3 -> GND
- RGB59 pad 3: 3V3 -> +5V
- RGB6 pad 1: 3V3 -> GND
- RGB6 pad 3: 3V3 -> +5V
- RGB60 pad 1: 3V3 -> GND
- RGB60 pad 3: 3V3 -> +5V
- RGB61 pad 1: 3V3 -> GND
- RGB61 pad 3: 3V3 -> +5V
- RGB62 pad 1: 3V3 -> GND
- RGB62 pad 3: 3V3 -> +5V
- RGB63 pad 1: 3V3 -> GND
- RGB63 pad 3: 3V3 -> +5V
- RGB64 pad 1: 3V3 -> GND
- RGB64 pad 3: 3V3 -> +5V
- RGB65 pad 1: 3V3 -> GND
- RGB65 pad 3: 3V3 -> +5V
- RGB66 pad 1: 3V3 -> GND
- RGB66 pad 3: 3V3 -> +5V
- RGB67 pad 1: 3V3 -> GND
- RGB67 pad 3: 3V3 -> +5V
- RGB68 pad 1: 3V3 -> GND
- RGB68 pad 3: 3V3 -> +5V
- RGB69 pad 1: 3V3 -> GND
- RGB69 pad 3: 3V3 -> +5V
- RGB7 pad 1: 3V3 -> GND
- RGB7 pad 3: 3V3 -> +5V
- RGB70 pad 1: 3V3 -> GND
- RGB70 pad 3: 3V3 -> +5V
- RGB71 pad 1: 3V3 -> GND
- RGB71 pad 3: 3V3 -> +5V
- RGB72 pad 1: 3V3 -> GND
- RGB72 pad 3: 3V3 -> +5V
- RGB73 pad 1: 3V3 -> GND
- RGB73 pad 3: 3V3 -> +5V
- RGB74 pad 1: 3V3 -> GND
- RGB74 pad 3: 3V3 -> +5V
- RGB75 pad 1: 3V3 -> GND
- RGB75 pad 3: 3V3 -> +5V
- RGB76 pad 1: 3V3 -> GND
- RGB76 pad 3: 3V3 -> +5V
- RGB77 pad 1: 3V3 -> GND
- RGB77 pad 3: 3V3 -> +5V
- RGB78 pad 1: 3V3 -> GND
- RGB78 pad 3: 3V3 -> +5V
- RGB79 pad 1: 3V3 -> GND
- RGB79 pad 3: 3V3 -> +5V
- RGB8 pad 1: 3V3 -> GND
- RGB8 pad 3: 3V3 -> +5V
- RGB80 pad 1: 3V3 -> GND
- RGB80 pad 3: 3V3 -> +5V
- RGB81 pad 1: 3V3 -> GND
- RGB81 pad 3: 3V3 -> +5V
- RGB82 pad 1: 3V3 -> GND
- RGB82 pad 3: 3V3 -> +5V
- RGB82 pad 4: unconnected-(RGB82-DOUT-Pad4) -> RGB_D82
- RGB83 pad 1: 3V3 -> GND
- RGB83 pad 2: RGB_57 -> RGB_D82
- RGB83 pad 3: 3V3 -> +5V
- RGB84 pad 1: 3V3 -> GND
- RGB84 pad 3: 3V3 -> +5V
- RGB84 pad 4: RGB_84 -> unconnected-(RGB84-DOUT-Pad4)
- RGB9 pad 1: 3V3 -> GND
- RGB9 pad 3: 3V3 -> +5V
Routing:
- net GND: track 0.00 -> 2519.8 mm, vias 0 -> 15
- net RGB_84: track 350.7 -> 0.00 mm, vias 2 -> 0
- net RGB_D57: track 0.00 -> 258.1 mm, vias 0 -> 2
- net 3V3: track 242.6 -> 0.00 mm, vias 47 -> 0
- net +5V: track 0.00 -> 170.6 mm, vias 0 -> 36
- net RGB_D82: track 0.00 -> 123.2 mm
- net RGB_57: track 52.4 -> 0.00 mm, vias 2 -> 0
- net /COL1: track 511.3 -> 506.3 mm
- net Net-(D91-A): track 16.2 -> 18.7 mm
- net /COL10: track 275.4 -> 273.0 mm
- net RGB_D58: track 42.2 -> 42.8 mm
- net RGB_D70: track 399.2 -> 399.9 mm, vias 2 -> 6
- net /ROW5: track 441.1 -> 441.6 mm
- added copper zone on B.Cu, net +5V
- removed copper zone on B.Cu, net 3V3
