File: my-keeb.kicad_sch (KiCad schematic)
At the start: 263 parts, among them SW10 SW_Push, SW11 SW_Push, SW12 SW_Push, SW13 SW_Push, SW14 SW_Push, SW15 SW_Push, SW16 SW_Push, SW17 SW_Push, SW18 SW_Push, SW19 SW_Push, SW2 SW_Push, SW20 SW_Push, SW21 SW_Push, SW22 SW_Push, SW23 SW_Push, SW24 SW_Push, SW25 SW_Push, SW26 SW_Push, SW27 SW_Push, SW29 SW_Push, SW3 SW_Push, SW30 SW_Push, SW31 SW_Push, SW32 SW_Push, SW33 SW_Push, SW34 SW_Push, SW35 SW_Push, SW36 SW_Push, SW37 SW_Push, SW38 SW_Push, SW39 SW_Push, SW4 SW_Push, SW40 SW_Push, SW41 SW_Push, SW42 SW_Push, SW43 SW_Push, SW44 SW_Push, SW45 SW_Push, SW46 SW_Push, SW47 SW_Push, SW48 SW_Push, SW49 SW_Push, SW5 SW_Push, SW50 SW_Push, SW51 SW_Push, SW52 SW_Push, SW53 SW_Push, SW54 SW_Push, SW55 SW_Push, SW57 SW_Push, SW58 SW_Push, SW6 SW_Push, SW60 SW_Push, SW61 SW_Push, SW62 SW_Push, SW63 SW_Push, SW64 SW_Push, SW65 SW_Push, SW66 SW_Push, SW67 SW_Push, SW68 SW_Push, SW69 SW_Push, SW7 SW_Push, SW71 SW_Push, SW72 SW_Push, SW73 SW_Push, SW74 SW_Push, SW77 SW_Push, SW79 SW_Push, SW8 SW_Push, SW80 SW_Push, SW81 SW_Push, SW82 SW_Push, SW86 SW_Push, SW87 SW_Push, SW88 SW_Push, SW89 SW_Push, SW9 SW_Push, SW90 SW_Push, SW91 SW_Push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

Commit message: Added mising connection for COL0
Connections:
- net RGB_14: now also U1.27 (GPA6)
- no-connect marks 22 -> 21
Changed lines of the file:
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@@
 	)
 	(no_connect
-		(at 199.39 139.7)
-	)
-	(no_connect
 		(at 173.99 142.24)
 	)
@@
 	(wire
 		(pts
+			(xy 102.87 182.88) (xy 113.03 182.88)
+		)
+		(stroke
+			(width 0)
+			(type default)
+		)
+	)
+	(wire
+		(pts
 			(xy 13.97 31.75) (xy 44.45 31.75)
 		)
@@
 	(wire
 		(pts
+			(xy 102.87 144.78) (xy 113.03 144.78)
+		)
+		(stroke
+			(width 0)
+			(type default)
+		)
+	)
+	(wire
+		(pts
 			(xy 196.85 99.06) (xy 196.85 100.33)
 		)
@@
 	(wire
 		(pts
+			(xy 102.87 170.18) (xy 113.03 170.18)
+		)
+		(stroke
+			(width 0)
+			(type default)
+		)
+	)
+	(wire
+		(pts
 			(xy 199.39 13.97) (xy 208.28 13.97)
 		)
@@
 	(wire
 		(pts
+			(xy 102.87 180.34) (xy 113.03 180.34)
+		)
+		(stroke
+			(width 0)
+			(type default)
+		)
+	)
+	(wire
+		(pts
 			(xy 146.05 92.71) (xy 158.75 92.71)
 		)
@@
 	(wire
 		(pts
+			(xy 102.87 177.8) (xy 113.03 177.8)
+		)
+		(stroke
+			(width 0)
+			(type default)
+		)
+	)
+	(wire
+		(pts
 			(xy 123.19 38.1) (xy 123.19 53.34)
 		)
@@
 	(wire
 		(pts
+			(xy 83.82 162.56) (xy 113.03 162.56)
+		)
+		(stroke
+			(width 0)
+			(type default)
+		)
+	)
+	(wire
+		(pts
 			(xy 13.97 46.99) (xy 44.45 46.99)
 		)
@@
 	(wire
 		(pts
+			(xy 199.39 139.7) (xy 204.47 139.7)
+		)
+		(stroke
+			(width 0)
+			(type default)
+		)
+	)
+	(wire
+		(pts
 			(xy 34.29 83.82) (xy 34.29 99.06)
 		)
@@
 	(wire
 		(pts
+			(xy 102.87 147.32) (xy 113.03 147.32)
+		)
+		(stroke
+			(width 0)
+			(type default)
+		)
+	)
+	(wire
+		(pts
 			(xy 44.45 22.86) (xy 44.45 24.13)
 		)
@@
 	(wire
 		(pts
+			(xy 102.87 154.94) (xy 113.03 154.94)
+		)
+		(stroke
+			(width 0)
+			(type default)
+		)
+	)
+	(wire
+		(pts
 			(xy 173.99 83.82) (xy 173.99 99.06)
 		)
@@
 	(wire
 		(pts
+			(xy 102.87 157.48) (xy 113.03 157.48)
+		)
+		(stroke
+			(width 0)
+			(type default)
+		)
+	)
+	(wire
+		(pts
 			(xy 148.59 22.86) (xy 148.59 38.1)
 		)
@@
 	(wire
 		(pts
+			(xy 102.87 152.4) (xy 113.03 152.4)
+		)
+		(stroke
+			(width 0)
+			(type default)
+		)
+	)
+	(wire
+		(pts
 			(xy 44.45 31.75) (xy 57.15 31.75)
 		)
@@
 	(wire
 		(pts
+			(xy 102.87 175.26) (xy 113.03 175.26)
+		)
+		(stroke
+			(width 0)
+			(type default)
+		)
+	)
+	(wire
+		(pts
 			(xy 184.15 83.82) (xy 184.15 85.09)
 		)
@@
 	(wire
 		(pts
+			(xy 102.87 172.72) (xy 113.03 172.72)
+		)
+		(stroke
+			(width 0)
+			(type default)
+		)
+	)
+	(wire
+		(pts
 			(xy 171.45 38.1) (xy 171.45 39.37)
 		)
@@
 	(wire
 		(pts
+			(xy 104.14 160.02) (xy 113.03 160.02)
+		)
+		(stroke
+			(width 0)
+			(type default)
+		)
+	)
+	(wire
+		(pts
 			(xy 72.39 68.58) (xy 72.39 83.82)
 		)
@@
 	(wire
 		(pts
+			(xy 102.87 167.64) (xy 113.03 167.64)
+		)
+		(stroke
+			(width 0)
+			(type default)
+		)
+	)
+	(wire
+		(pts
 			(xy 148.59 68.58) (xy 148.59 83.82)
 		)
@@
 	(wire
 		(pts
+			(xy 102.87 149.86) (xy 113.03 149.86)
+		)
+		(stroke
+			(width 0)
+			(type default)
+		)
+	)
+	(wire
+		(pts
 			(xy 240.03 83.82) (xy 240.03 85.09)
 		)
@@
 	(wire
 		(pts
+			(xy 102.87 165.1) (xy 113.03 165.1)
+		)
+		(stroke
+			(width 0)
+			(type default)
+		)
+	)
+	(wire
+		(pts
 			(xy 252.73 53.34) (xy 252.73 54.61)
 		)
@@
 	)
 	(label "COL2"
-		(at 113.03 165.1 0)
+		(at 102.87 165.1 0)
 		(effects
 			(font
@@
 	)
 	(label "COL4"
-		(at 113.03 170.18 0)
+		(at 102.87 170.18 0)
 		(effects
 			(font
@@
 	)
 	(label "ROW2"
-		(at 113.03 149.86 0)
+		(at 102.87 149.86 0)
 		(effects
 			(font
@@
 	)
 	(label "ROW1"
-		(at 113.03 147.32 0)
+		(at 102.87 147.32 0)
 		(effects
 			(font
@@
 	)
 	(label "COL3"
-		(at 113.03 167.64 0)
+		(at 102.87 167.64 0)
 		(effects
 			(font
@@
 	)
 	(label "ROW4"
-		(at 113.03 154.94 0)
+		(at 102.87 154.94 0)
 		(effects
 			(font
@@
 	)
 	(label "COL7"
-		(at 113.03 177.8 0)
+		(at 102.87 177.8 0)
 		(effects
 			(font
@@
 		)
 	)
+	(label "COL1"
+		(at 204.47 139.7 0)
+		(effects
+			(font
+				(size 1.27 1.27)
+			)
+			(justify left bottom)
+		)
+	)
 	(label "COL12"
 		(at 195.58 13.97 0)
@@
 	)
 	(label "ROW0"
-		(at 113.03 144.78 0)
+		(at 102.87 144.78 0)
 		(effects
 			(font
@@
 	)
 	(label "COL6"
-		(at 113.03 175.26 0)
+		(at 102.87 175.26 0)
 		(effects
 			(font
@@
 	)
 	(label "ROW5"
-		(at 113.03 157.48 0)
+		(at 102.87 157.48 0)
 		(effects
 			(font
@@
 	)
 	(label "COL8"
-		(at 113.03 180.34 0)
+		(at 102.87 180.34 0)
 		(effects
 			(font
@@
 	)
 	(label "ROW3"
-		(at 113.03 152.4 0)
+		(at 102.87 152.4 0)
 		(effects
 			(font
@@
 	)
 	(label "COL0"
-		(at 113.03 160.02 0)
+		(at 104.14 160.02 0)
 		(effects
 			(font
@@
 	)
 	(label "COL9"
-		(at 113.03 182.88 0)
+		(at 102.87 182.88 0)
 		(effects
 			(font
@@
 	)
 	(label "COL5"
-		(at 113.03 172.72 0)
+		(at 102.87 172.72 0)
 		(effects
 			(font
@@
 	(global_label "RGB_DATA"
 		(shape bidirectional)
-		(at 113.03 162.56 0)
+		(at 83.82 162.56 0)
 		(effects
 			(font
@@
 		)
 		(property "Intersheetrefs" "${INTERSHEET_REFS}"
-			(at 113.03 162.56 0)
+			(at 83.82 162.56 0)
 			(hide yes)
 			(show_name no)

Commit message: Add files via upload
Parts:
- removed C1: 100nF, Capacitor_SMD:C_0603_1608Metric, symbol Device:C
- removed R1, R2: 4.7k, Resistor_SMD:R_0603_1608Metric, symbol Device:R
- removed U1: MCP23017x-x-SO, Package_SO:SOIC-28W_7.5x17.9mm_P1.27mm, symbol Interface_Expansion:MCP23017x-x-SO
- added D1, D28: 1N4148, Diode_THT:D_DO-35_SOD27_P7.62mm_Horizontal, symbol Diode:1N4148
Connections:
- net I2C_SCL is gone; now on net ENC1_A: A1.32 (GPIO27_ADC1)
- net I2C_SDA is gone; now on net RGB_DATA: A1.31 (GPIO26_ADC0)
- net MCP23017_INT is gone; now on net ENC1_B: A1.34 (GPIO28_ADC2)
- net 3V3: now also A1.13 (GND), A1.18 (GND), A1.23 (GND), A1.28 (GND), A1.3 (GND), A1.38 (GND), A1.8 (GND); no longer A1.27 (GPIO21), SW86.1, SW91.1, SW95.1
- net ENC2_A: now also A1.27 (GPIO21)
- net ENC2_B: now also A1.29 (GPIO22)
- net RGB_14: now also A1.10 (GPIO7), SW87.1
- net RGB_16: now also SW91.1
- net RGB_17: now also SW92.1
- net RGB_25: now also SW86.1, SW89.1, SW95.1
- net RGB_27: no longer A1.29 (GPIO22), RGB43.4 (DOUT), RGB44.2 (DIN), RGB70.4 (DOUT), RGB71.2 (DIN), SW87.1, SW89.1, SW92.1
- net RGB_DATA: no longer A1.10 (GPIO7)
- net ROW0: now also D28.1 (K)
- net ROW1: now also D1.1 (K); no longer D87.1 (K)
- net ROW2: no longer D89.1 (K)
- net ROW4: now also D87.1 (K), D89.1 (K)
- net ENC1_SW: no longer names the net of ENC1.S1
- net ENC1_SW: now also D28.2 (A)
- net ENC2_SW: no longer names the net of ENC2.S1
- net ENC2_SW: now also D1.2 (A)
- net Net-(D15-A): no longer names the net of D15.2 (A), SW15.2
- new net RGB_43: RGB43.4 (DOUT), RGB44.2 (DIN)
- new net RGB_70: RGB70.4 (DOUT), RGB71.2 (DIN)
- no-connect marks 21 -> 7
Other:
- moved on the sheet: ENC2

Commit message: Add files via upload
Parts:
- added S8: MX_stab_6.25u, my-keeb:STAB_MX_P_6.25u, symbol PCM_marbastlib-mx:MX_stab
Connections:
- net +5V: now reaches A1.40 (VBUS)
- net +5V: now also RGB1.3 (VDD), RGB10.3 (VDD), RGB11.3 (VDD), RGB12.3 (VDD), RGB13.3 (VDD), RGB14.3 (VDD), RGB15.3 (VDD), RGB16.3 (VDD), RGB17.3 (VDD), RGB18.3 (VDD), RGB19.3 (VDD), RGB2.3 (VDD), RGB20.3 (VDD), RGB21.3 (VDD), RGB22.3 (VDD), RGB23.3 (VDD), RGB24.3 (VDD), RGB25.3 (VDD), RGB26.3 (VDD), RGB27.3 (VDD), RGB28.3 (VDD), RGB29.3 (VDD), RGB3.3 (VDD), RGB30.3 (VDD), RGB31.3 (VDD), RGB32.3 (VDD), RGB33.3 (VDD), RGB34.3 (VDD), RGB35.3 (VDD), RGB36.3 (VDD), RGB37.3 (VDD), RGB38.3 (VDD), RGB39.3 (VDD), RGB4.3 (VDD), RGB40.3 (VDD), RGB41.3 (VDD), RGB42.3 (VDD), RGB43.3 (VDD), RGB44.3 (VDD), RGB45.3 (VDD), RGB46.3 (VDD), RGB47.3 (VDD), RGB48.3 (VDD), RGB49.3 (VDD), RGB5.3 (VDD), RGB50.3 (VDD), RGB51.3 (VDD), RGB52.3 (VDD), RGB53.3 (VDD), RGB54.3 (VDD), RGB55.3 (VDD), RGB56.3 (VDD), RGB57.3 (VDD), RGB58.3 (VDD), RGB59.3 (VDD), RGB6.3 (VDD), RGB60.3 (VDD), RGB61.3 (VDD), RGB62.3 (VDD), RGB63.3 (VDD), RGB64.3 (VDD), RGB65.3 (VDD), RGB66.3 (VDD), RGB67.3 (VDD), RGB68.3 (VDD), RGB69.3 (VDD), RGB7.3 (VDD), RGB70.3 (VDD), RGB71.3 (VDD), RGB72.3 (VDD), RGB73.3 (VDD), RGB74.3 (VDD), RGB75.3 (VDD), RGB76.3 (VDD), RGB77.3 (VDD), RGB78.3 (VDD), RGB79.3 (VDD), RGB8.3 (VDD), RGB80.3 (VDD), RGB81.3 (VDD), RGB82.3 (VDD), RGB83.3 (VDD), RGB84.3 (VDD), RGB9.3 (VDD)
- net RGB_D82: now reaches RGB82.4 (DOUT)
- net RGB_D82: now also RGB83.2 (DIN)
- net 3V3 renamed GND
- net GND: no longer A1.26 (GPIO20), A1.36 (3V3), ENC1.S2, ENC2.S2, RGB1.3 (VDD), RGB10.3 (VDD), RGB11.3 (VDD), RGB12.3 (VDD), RGB13.3 (VDD), RGB14.3 (VDD), RGB15.3 (VDD), RGB16.3 (VDD), RGB17.3 (VDD), RGB18.3 (VDD), RGB19.3 (VDD), RGB2.3 (VDD), RGB20.3 (VDD), RGB21.3 (VDD), RGB22.3 (VDD), RGB23.3 (VDD), RGB24.3 (VDD), RGB25.3 (VDD), RGB26.3 (VDD), RGB27.3 (VDD), RGB28.3 (VDD), RGB29.3 (VDD), RGB3.3 (VDD), RGB30.3 (VDD), RGB31.3 (VDD), RGB32.3 (VDD), RGB33.3 (VDD), RGB34.3 (VDD), RGB35.3 (VDD), RGB36.3 (VDD), RGB37.3 (VDD), RGB38.3 (VDD), RGB39.3 (VDD), RGB4.3 (VDD), RGB40.3 (VDD), RGB41.3 (VDD), RGB42.3 (VDD), RGB43.3 (VDD), RGB44.3 (VDD), RGB45.3 (VDD), RGB46.3 (VDD), RGB47.3 (VDD), RGB48.3 (VDD), RGB49.3 (VDD), RGB5.3 (VDD), RGB50.3 (VDD), RGB51.3 (VDD), RGB52.3 (VDD), RGB53.3 (VDD), RGB54.3 (VDD), RGB55.3 (VDD), RGB56.3 (VDD), RGB57.3 (VDD), RGB58.3 (VDD), RGB59.3 (VDD), RGB6.3 (VDD), RGB60.3 (VDD), RGB61.3 (VDD), RGB62.3 (VDD), RGB63.3 (VDD), RGB64.3 (VDD), RGB65.3 (VDD), RGB66.3 (VDD), RGB67.3 (VDD), RGB68.3 (VDD), RGB69.3 (VDD), RGB7.3 (VDD), RGB70.3 (VDD), RGB71.3 (VDD), RGB72.3 (VDD), RGB73.3 (VDD), RGB74.3 (VDD), RGB75.3 (VDD), RGB76.3 (VDD), RGB77.3 (VDD), RGB78.3 (VDD), RGB79.3 (VDD), RGB8.3 (VDD), RGB80.3 (VDD), RGB81.3 (VDD), RGB82.3 (VDD), RGB83.3 (VDD), RGB84.3 (VDD), RGB9.3 (VDD), SW88.1, SW90.1, SW93.1, SW94.1
- removed net RGB_1: A1.20 (GPIO15), RGB1.4 (DOUT), RGB2.2 (DIN), RGB22.4 (DOUT), RGB23.2 (DIN), RGB37.4 (DOUT), RGB38.2 (DIN), RGB53.4 (DOUT), RGB54.2 (DIN), SW11.1, SW25.1, SW39.1, SW53.1, SW67.1
- removed net RGB_10: A1.15 (GPIO11), RGB10.4 (DOUT), RGB11.2 (DIN), RGB18.4 (DOUT), RGB19.2 (DIN), RGB33.4 (DOUT), RGB34.2 (DIN), RGB49.4 (DOUT), RGB50.2 (DIN), SW21.1, SW35.1, SW49.1, SW63.1, SW7.1
- removed net RGB_11: A1.16 (GPIO12), RGB11.4 (DOUT), RGB12.2 (DIN), RGB19.4 (DOUT), RGB20.2 (DIN), RGB34.4 (DOUT), RGB35.2 (DIN), RGB50.4 (DOUT), RGB51.2 (DIN), SW22.1, SW36.1, SW50.1, SW64.1, SW8.1
- removed net RGB_12: A1.17 (GPIO13), RGB12.4 (DOUT), RGB13.2 (DIN), RGB20.4 (DOUT), RGB21.2 (DIN), RGB35.4 (DOUT), RGB36.2 (DIN), RGB51.4 (DOUT), RGB52.2 (DIN), RGB63.4 (DOUT), RGB64.2 (DIN), SW23.1, SW37.1, SW51.1, SW65.1, SW77.1, SW9.1
- removed net RGB_13: A1.19 (GPIO14), RGB13.4 (DOUT), RGB14.2 (DIN), RGB21.4 (DOUT), RGB22.2 (DIN), RGB36.4 (DOUT), RGB37.2 (DIN), RGB52.4 (DOUT), RGB53.2 (DIN), SW10.1, SW24.1, SW38.1, SW52.1, SW66.1
- removed net RGB_14: A1.10 (GPIO7), RGB14.4 (DOUT), RGB15.2 (DIN), RGB29.4 (DOUT), RGB30.2 (DIN), RGB45.4 (DOUT), RGB46.2 (DIN), RGB58.4 (DOUT), RGB59.2 (DIN), RGB6.4 (DOUT), RGB7.2 (DIN), SW17.1, SW3.1, SW31.1, SW45.1, SW73.1, SW87.1
- removed net RGB_15: A1.11 (GPIO8), RGB15.4 (DOUT), RGB16.2 (DIN), RGB30.4 (DOUT), RGB31.2 (DIN), RGB46.4 (DOUT), RGB47.2 (DIN), RGB7.4 (DOUT), RGB8.2 (DIN), SW18.1, SW32.1, SW4.1, SW46.1, SW60.1, SW74.1
- removed net RGB_16: A1.12 (GPIO9), RGB16.4 (DOUT), RGB17.2 (DIN), RGB31.4 (DOUT), RGB32.2 (DIN), RGB47.4 (DOUT), RGB48.2 (DIN), RGB8.4 (DOUT), RGB9.2 (DIN), SW19.1, SW33.1, SW47.1, SW5.1, SW61.1, SW91.1
- removed net RGB_17: A1.14 (GPIO10), RGB10.2 (DIN), RGB17.4 (DOUT), RGB18.2 (DIN), RGB32.4 (DOUT), RGB33.2 (DIN), RGB48.4 (DOUT), RGB49.2 (DIN), RGB9.4 (DOUT), SW20.1, SW34.1, SW48.1, SW6.1, SW62.1, SW92.1
- removed net RGB_2: A1.21 (GPIO16), RGB2.4 (DOUT), RGB23.4 (DOUT), RGB24.2 (DIN), RGB3.2 (DIN), RGB38.4 (DOUT), RGB39.2 (DIN), RGB54.4 (DOUT), RGB55.2 (DIN), RGB66.4 (DOUT), RGB67.2 (DIN), SW12.1, SW26.1, SW40.1, SW54.1, SW68.1, SW79.1
- removed net RGB_24: A1.22 (GPIO17), RGB24.4 (DOUT), RGB25.2 (DIN), RGB3.4 (DOUT), RGB39.4 (DOUT), RGB4.2 (DIN), RGB40.2 (DIN), RGB55.4 (DOUT), RGB56.2 (DIN), RGB67.4 (DOUT), RGB68.2 (DIN), SW13.1, SW27.1, SW41.1, SW55.1, SW69.1, SW80.1
- removed net RGB_25: A1.24 (GPIO18), RGB25.4 (DOUT), RGB26.2 (DIN), RGB4.4 (DOUT), RGB40.4 (DOUT), RGB41.2 (DIN), RGB5.2 (DIN), RGB56.4 (DOUT), RGB57.2 (DIN), RGB68.4 (DOUT), RGB69.2 (DIN), SW14.1, SW42.1, SW81.1, SW86.1, SW89.1, SW95.1
- net RGB_26 renamed RGB_D26
- net RGB_27 renamed RGB_D27
- net RGB_28 renamed RGB_D28
- net RGB_41 renamed COL13
- net COL13: no longer RGB41.4 (DOUT), RGB42.2 (DIN), RGB5.4 (DOUT), RGB6.2 (DIN)
- net RGB_42 renamed RGB_D42
- net RGB_43 renamed RGB_D43
- net RGB_44 renamed RGB_D44
- net RGB_57 renamed RGB_D57
- net RGB_D57: now also RGB58.2 (DIN); no longer RGB83.2 (DIN)
- net RGB_59 renamed RGB_D59
- net RGB_60 renamed RGB_D60
- net RGB_61 renamed RGB_D61
- net RGB_62 renamed RGB_D62
- net RGB_64 renamed RGB_D64
- net RGB_65 renamed RGB_D65
- net RGB_69 renamed RGB_D69
- net RGB_70 renamed RGB_D70
- net RGB_71 renamed RGB_D71
- net RGB_72 renamed RGB_D72
- net RGB_73 renamed RGB_D73
- net RGB_74 renamed RGB_D74
- net RGB_75 renamed RGB_D75
- net RGB_76 renamed RGB_D76
- net RGB_77 renamed RGB_D77
- net RGB_78 renamed RGB_D78
- net RGB_79 renamed RGB_D79
- net RGB_80 renamed RGB_D80
- net RGB_81 renamed RGB_D81
- net RGB_83 renamed RGB_D83
- net RGB_84: no longer names the net of RGB84.4 (DOUT)
- net RGB_84: no longer RGB58.2 (DIN)
- new net COL1: A1.10 (GPIO7), SW17.1, SW3.1, SW31.1, SW45.1, SW73.1, SW87.1
- new net COL10: A1.21 (GPIO16), SW12.1, SW26.1, SW40.1, SW54.1, SW68.1, SW79.1
- new net COL11: A1.22 (GPIO17), SW13.1, SW27.1, SW41.1, SW55.1, SW69.1, SW80.1
- new net COL12: A1.24 (GPIO18), SW14.1, SW42.1, SW81.1, SW86.1, SW89.1, SW95.1
- new net COL14: A1.26 (GPIO20), ENC1.S2, ENC2.S2, SW88.1, SW90.1, SW93.1, SW94.1
- new net COL2: A1.11 (GPIO8), SW18.1, SW32.1, SW4.1, SW46.1, SW60.1, SW74.1
- new net COL3: A1.12 (GPIO9), SW19.1, SW33.1, SW47.1, SW5.1, SW61.1, SW91.1
- new net COL4: A1.14 (GPIO10), SW20.1, SW34.1, SW48.1, SW6.1, SW62.1, SW92.1
- new net COL5: A1.15 (GPIO11), SW21.1, SW35.1, SW49.1, SW63.1, SW7.1
- new net COL6: A1.16 (GPIO12), SW22.1, SW36.1, SW50.1, SW64.1, SW8.1
- new net COL7: A1.17 (GPIO13), SW23.1, SW37.1, SW51.1, SW65.1, SW77.1, SW9.1
- new net COL8: A1.19 (GPIO14), SW10.1, SW24.1, SW38.1, SW52.1, SW66.1
- new net COL9: A1.20 (GPIO15), SW11.1, SW25.1, SW39.1, SW53.1, SW67.1
- new net RGB_D1: RGB1.4 (DOUT), RGB2.2 (DIN)
- new net RGB_D10: RGB10.4 (DOUT), RGB11.2 (DIN)
- new net RGB_D11: RGB11.4 (DOUT), RGB12.2 (DIN)
- new net RGB_D12: RGB12.4 (DOUT), RGB13.2 (DIN)
- new net RGB_D13: RGB13.4 (DOUT), RGB14.2 (DIN)
- new net RGB_D14: RGB14.4 (DOUT), RGB15.2 (DIN)
- new net RGB_D15: RGB15.4 (DOUT), RGB16.2 (DIN)
- new net RGB_D16: RGB16.4 (DOUT), RGB17.2 (DIN)
- new net RGB_D17: RGB17.4 (DOUT), RGB18.2 (DIN)
- new net RGB_D18: RGB18.4 (DOUT), RGB19.2 (DIN)
- new net RGB_D19: RGB19.4 (DOUT), RGB20.2 (DIN)
- new net RGB_D2: RGB2.4 (DOUT), RGB3.2 (DIN)
- new net RGB_D20: RGB20.4 (DOUT), RGB21.2 (DIN)
- new net RGB_D21: RGB21.4 (DOUT), RGB22.2 (DIN)
- new net RGB_D22: RGB22.4 (DOUT), RGB23.2 (DIN)
- new net RGB_D23: RGB23.4 (DOUT), RGB24.2 (DIN)
- new net RGB_D24: RGB24.4 (DOUT), RGB25.2 (DIN)
- new net RGB_D25: RGB25.4 (DOUT), RGB26.2 (DIN)
- new net RGB_D29: RGB29.4 (DOUT), RGB30.2 (DIN)
- new net RGB_D3: RGB3.4 (DOUT), RGB4.2 (DIN)
- new net RGB_D30: RGB30.4 (DOUT), RGB31.2 (DIN)
- new net RGB_D31: RGB31.4 (DOUT), RGB32.2 (DIN)
- new net RGB_D32: RGB32.4 (DOUT), RGB33.2 (DIN)
- new net RGB_D33: RGB33.4 (DOUT), RGB34.2 (DIN)
- new net RGB_D34: RGB34.4 (DOUT), RGB35.2 (DIN)
- new net RGB_D35: RGB35.4 (DOUT), RGB36.2 (DIN)
- new net RGB_D36: RGB36.4 (DOUT), RGB37.2 (DIN)
- new net RGB_D37: RGB37.4 (DOUT), RGB38.2 (DIN)
- new net RGB_D38: RGB38.4 (DOUT), RGB39.2 (DIN)
- new net RGB_D39: RGB39.4 (DOUT), RGB40.2 (DIN)
- new net RGB_D4: RGB4.4 (DOUT), RGB5.2 (DIN)
- new net RGB_D40: RGB40.4 (DOUT), RGB41.2 (DIN)
- new net RGB_D41: RGB41.4 (DOUT), RGB42.2 (DIN)
- new net RGB_D45: RGB45.4 (DOUT), RGB46.2 (DIN)
- new net RGB_D46: RGB46.4 (DOUT), RGB47.2 (DIN)
- new net RGB_D47: RGB47.4 (DOUT), RGB48.2 (DIN)
- new net RGB_D48: RGB48.4 (DOUT), RGB49.2 (DIN)
- new net RGB_D49: RGB49.4 (DOUT), RGB50.2 (DIN)
- new net RGB_D5: RGB5.4 (DOUT), RGB6.2 (DIN)
- new net RGB_D50: RGB50.4 (DOUT), RGB51.2 (DIN)
- new net RGB_D51: RGB51.4 (DOUT), RGB52.2 (DIN)
- new net RGB_D52: RGB52.4 (DOUT), RGB53.2 (DIN)
- new net RGB_D53: RGB53.4 (DOUT), RGB54.2 (DIN)
- new net RGB_D54: RGB54.4 (DOUT), RGB55.2 (DIN)
- new net RGB_D55: RGB55.4 (DOUT), RGB56.2 (DIN)
- new net RGB_D56: RGB56.4 (DOUT), RGB57.2 (DIN)
- new net RGB_D58: RGB58.4 (DOUT), RGB59.2 (DIN)
- new net RGB_D6: RGB6.4 (DOUT), RGB7.2 (DIN)
- new net RGB_D63: RGB63.4 (DOUT), RGB64.2 (DIN)
- new net RGB_D66: RGB66.4 (DOUT), RGB67.2 (DIN)
- new net RGB_D67: RGB67.4 (DOUT), RGB68.2 (DIN)
- new net RGB_D68: RGB68.4 (DOUT), RGB69.2 (DIN)
- new net RGB_D7: RGB7.4 (DOUT), RGB8.2 (DIN)
- new net RGB_D8: RGB8.4 (DOUT), RGB9.2 (DIN)
- new net RGB_D9: RGB10.2 (DIN), RGB9.4 (DOUT)
Other:
- moved on the sheet: RGB1, RGB10, RGB11, RGB12, RGB13, RGB14, RGB15, RGB16, RGB17, RGB18, RGB19, RGB2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
