File: Kicad/my-keeb.kicad_pcb (KiCad board)
At the start: 2 copper layers, 355.7 x 122 mm, 262 parts, among them SW10 SW_Push, SW11 SW_Push, SW12 SW_Push, SW13 SW_Push, SW14 SW_Push, SW15 SW_Push, SW16 SW_Push, SW17 SW_Push, SW18 SW_Push, SW19 SW_Push, SW2 SW_Push, SW20 SW_Push, SW21 SW_Push, SW22 SW_Push, SW23 SW_Push, SW24 SW_Push, SW25 SW_Push, SW26 SW_Push, SW27 SW_Push, SW29 SW_Push, SW3 SW_Push, SW30 SW_Push, SW31 SW_Push, SW32 SW_Push, SW33 SW_Push, SW34 SW_Push, SW35 SW_Push, SW36 SW_Push, SW37 SW_Push, SW38 SW_Push, SW39 SW_Push, SW4 SW_Push, SW40 SW_Push, SW41 SW_Push, SW42 SW_Push, SW43 SW_Push, SW44 SW_Push, SW45 SW_Push, SW46 SW_Push, SW47 SW_Push, SW48 SW_Push, SW49 SW_Push, SW5 SW_Push, SW50 SW_Push, SW51 SW_Push, SW52 SW_Push, SW53 SW_Push, SW54 SW_Push, SW55 SW_Push, SW57 SW_Push, SW58 SW_Push, SW6 SW_Push, SW60 SW_Push, SW61 SW_Push, SW62 SW_Push, SW63 SW_Push, SW64 SW_Push, SW65 SW_Push, SW66 SW_Push, SW67 SW_Push, SW68 SW_Push, SW69 SW_Push, SW7 SW_Push, SW71 SW_Push, SW72 SW_Push, SW73 SW_Push, SW74 SW_Push, SW77 SW_Push, SW79 SW_Push, SW8 SW_Push, SW80 SW_Push, SW81 SW_Push, SW82 SW_Push, SW86 SW_Push, SW87 SW_Push, SW88 SW_Push, SW89 SW_Push, SW9 SW_Push, SW90 SW_Push, SW91 SW_Push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

Commit message: Organize files into folders
Routing:
- net +5V: track 170.6 -> 236.2 mm, vias 36 -> 44
Changed lines of the file:
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@@
+	)
+	(segment
+		(start 317 117)
+		(end 318.25 115.75)
+		(width 0.2)
+		(layer "F.Cu")
+		(net "+5V")
 	)
 	(segment
@@
 	)
 	(segment
+		(start 42 50.25)
+		(end 42 32.25)
+		(width 0.2)
+		(layer "F.Cu")
+		(net "+5V")
+	)
+	(segment
 		(start 234 137.5)
 		(end 236.25 137.5)
@@
 	)
 	(segment
-		(start 313.5 121.25)
-		(end 308.75 126)
+		(start 312.25 122.5)
+		(end 310.25 124.5)
 		(width 0.2)
 		(layer "F.Cu")
@@
 	)
 	(segment
+		(start 42 30.25)
+		(end 42 32.25)
+		(width 0.2)
+		(layer "F.Cu")
+		(net "+5V")
+	)
+	(segment
 		(start 182.25 108.5)
 		(end 182.25 94.5)
@@
 	)
 	(segment
+		(start 35.5 54.25)
+		(end 38 54.25)
+		(width 0.2)
+		(layer "F.Cu")
+		(net "+5V")
+	)
+	(segment
+		(start 35.5 54.25)
+		(end 35.5 70.25)
+		(width 0.2)
+		(layer "F.Cu")
+		(net "+5V")
+	)
+	(segment
+		(start 42 32.25)
+		(end 42 33.25)
+		(width 0.2)
+		(layer "F.Cu")
+		(net "+5V")
+	)
+	(segment
+		(start 312.25 129)
+		(end 313.25 130)
+		(width 0.2)
+		(layer "F.Cu")
+		(net "+5V")
+	)
+	(segment
 		(start 182.25 94.5)
 		(end 177.5 89.75)
@@
 	)
 	(segment
+		(start 35.5 70.25)
+		(end 36.5 71.25)
+		(width 0.2)
+		(layer "F.Cu")
+		(net "+5V")
+	)
+	(segment
 		(start 345.75 121.5)
 		(end 345.75 119.5)
@@
 	)
 	(segment
+		(start 314.25 117)
+		(end 317 117)
+		(width 0.2)
+		(layer "F.Cu")
+		(net "+5V")
+	)
+	(segment
+		(start 313.5 121.25)
+		(end 312.25 122.5)
+		(width 0.2)
+		(layer "F.Cu")
+		(net "+5V")
+	)
+	(segment
 		(start 363.77 84.75)
 		(end 364 84.52)
@@
 	)
 	(segment
+		(start 310.25 124.5)
+		(end 308.75 126)
+		(width 0.2)
+		(layer "F.Cu")
+		(net "+5V")
+	)
+	(segment
+		(start 38 54.25)
+		(end 42 50.25)
+		(width 0.2)
+		(layer "F.Cu")
+		(net "+5V")
+	)
+	(segment
 		(start 294 138)
 		(end 294 141)
@@
 	)
 	(segment
+		(start 312.25 122.5)
+		(end 312.25 129)
+		(width 0.2)
+		(layer "F.Cu")
+		(net "+5V")
+	)
+	(segment
 		(start 211.25 139.25)
 		(end 211.25 125)
@@
 		(net "+5V")
 	)
+	(segment
+		(start 33.5 54.25)
+		(end 35.5 54.25)
+		(width 0.2)
+		(layer "F.Cu")
+		(net "+5V")
+	)
 	(via
 		(at 345.25 114.75)
@@
 	)
 	(via
+		(at 313.25 130)
+		(size 0.6)
+		(drill 0.3)
+		(layers "F.Cu" "B.Cu")
+		(net "+5V")
+	)
+	(via
 		(at 363.77 84.75)
 		(size 0.6)
@@
 	)
 	(via
+		(at 36.5 71.25)
+		(size 0.6)
+		(drill 0.3)
+		(layers "F.Cu" "B.Cu")
+		(net "+5V")
+	)
+	(via
 		(at 278.5 139)
 		(size 0.6)
@@
 	)
 	(via
+		(at 318.25 115.75)
+		(size 0.6)
+		(drill 0.3)
+		(layers "F.Cu" "B.Cu")
+		(net "+5V")
+	)
+	(via
+		(at 33.5 54.25)
+		(size 0.6)
+		(drill 0.3)
+		(layers "F.Cu" "B.Cu")
+		(net "+5V")
+	)
+	(via
 		(at 278.5 142)
 		(size 0.6)
@@
 	)
 	(via
+		(at 314.25 117)
+		(size 0.6)
+		(drill 0.3)
+		(layers "F.Cu" "B.Cu")
+		(net "+5V")
+	)
+	(via
 		(at 56.75 138)
 		(size 0.6)
@@
 	)
 	(via
+		(at 310.25 124.5)
+		(size 0.6)
+		(drill 0.3)
+		(layers "F.Cu" "B.Cu")
+		(net "+5V")
+	)
+	(via
 		(at 345.25 108)
 		(size 0.6)
@@
 	)
 	(via
+		(at 42 33.25)
+		(size 0.6)
+		(drill 0.3)
+		(layers "F.Cu" "B.Cu")
+		(net "+5V")
+	)
+	(via
 		(at 16.5 102.75)
 		(size 0.6)
@@
 	(via
 		(at 229 141.25)
+		(size 0.6)
+		(drill 0.3)
+		(layers "F.Cu" "B.Cu")
+		(net "+5V")
+	)
+	(via
+		(at 42 30.25)
 		(size 0.6)
 		(drill 0.3)
@@
 	)
 	(segment
+		(start 314.25 120.5)
+		(end 314.25 117)
+		(width 0.2)
+		(layer "B.Cu")
+		(net "+5V")
+	)
+	(segment
 		(start 278.5 139)
 		(end 278.5 138.5)
 		(width 0.2)
 		(layer "B.Cu")
+		(net "+5V")
+	)
+	(segment
+		(start 313.5 121.25)
+		(end 314.25 120.5)
+		(width 0.2)
+		(layer "B.Cu")
